File: BeamRider_MainBoard_v1.kicad_pcb (KiCad board)
At the start: 2 copper layers, 246.5 x 120 mm, 24 parts, among them U1 RPR-220, U2 RPR-220, U3 RPR-220, U4 RPR-220, U5 RPR-220, U6 RPR-220, U7 RPR-220, U8 RPR-220, U9 RPR-220

Commit message: project structure
Parts:
- added MCU1: STM32F407VETx, Package_QFP:LQFP-100_14x14mm_P0.5mm, F.Cu at (136.0, 84.0)

Commit message: components selection
Parts:
- added BT1: LiION_18650, Battery:BatteryHolder_Keystone_1042_1x18650, F.Cu at (93.5, 82.5)
- added BT2: LiION_18650, Battery:BatteryHolder_Keystone_1042_1x18650, F.Cu at (72.0, 82.5)
- added C1: 100n 50V, Capacitor_SMD:C_0603_1608Metric_Pad1.08x0.95mm_HandSolder, F.Cu at (232.7, -59.1)
- added C2: 100n 50V, Capacitor_SMD:C_0603_1608Metric, F.Cu at (109.0, 14.5)
- added C3: 100n 50V, Capacitor_SMD:C_0603_1608Metric, F.Cu at (113.4, 12.6)
- added C4: 100n 50V, Capacitor_SMD:C_0603_1608Metric, F.Cu at (137.6, -6.62)
- added C5: 4.7u 10V, Capacitor_SMD:C_0805_2012Metric, F.Cu at (153.6, -13.4)
- added C6: 100n 50V, Capacitor_SMD:C_0603_1608Metric, F.Cu at (133.6, -6.62)
- added C7: 100n 50V, Capacitor_SMD:C_0603_1608Metric, F.Cu at (146.6, -9.13)
- added C8: 4.7u 10V, Capacitor_SMD:C_0805_2012Metric, F.Cu at (158.1, -13.4)
- added D1: TVS, Diode_SMD:D_SMA, F.Cu at (131.3, -12.7)
- added D2: TVS, Diode_SMD:D_SMA, F.Cu at (147.4, -12.7)
- added D3: 5.1V, Diode_SMD:D_SMA, F.Cu at (139.3, -12.7)
- added D4: LED G, LED_SMD:LED_0603_1608Metric_Pad1.05x0.95mm_HandSolder, F.Cu at (162.5, -13.6)
- added F1: 5A SLOW, Fuse:Fuse_1206_3216Metric_Pad1.42x1.75mm_HandSolder, F.Cu at (105.9, 1.20)
- added F2: 5A SLOW, Fuse:Fuse_1206_3216Metric_Pad1.42x1.75mm_HandSolder, F.Cu at (111.9, 1.20)
- added J1: Barrel_Jack, Connector_BarrelJack:BarrelJack_GCT_DCJ200-10-A_Horizontal, F.Cu at (103.1, 124.4)
- added J2: BATTERY_OUT, TerminalBlock:TerminalBlock_bornier-2_P5.08mm, F.Cu at (131.0, 125.3)
- added Q1: PMOS, Package_TO_SOT_SMD:TO-252-2, F.Cu at (109.0, -10.9)
- added Q2: PMOS, Package_TO_SOT_SMD:TO-252-2, F.Cu at (121.2, -10.9)
- added Q3: PMOS, Package_TO_SOT_SMD:TO-252-2, F.Cu at (197.6, -39.6)
- added R1: 47k 1%, Resistor_SMD:R_0603_1608Metric, F.Cu at (104.9, 14.5)
- added R2: 1Meg 1%, Resistor_SMD:R_0603_1608Metric_Pad0.98x0.95mm_HandSolder, F.Cu at (153.6, -10.7)
- added R3: 1Meg 1%, Resistor_SMD:R_0603_1608Metric_Pad0.98x0.95mm_HandSolder, F.Cu at (142.5, -9.13)
- added R4: 10k 1%, Resistor_SMD:R_0603_1608Metric_Pad0.98x0.95mm_HandSolder, F.Cu at (162.5, -11.1)
- added R5: 10k 1%, Resistor_SMD:R_0603_1608Metric_Pad0.98x0.95mm_HandSolder, F.Cu at (133.8, -9.13)
- added R6: 10k 1%, Resistor_SMD:R_0603_1608Metric_Pad0.98x0.95mm_HandSolder, F.Cu at (138.1, -9.13)
- added R7: 100R 1%, Resistor_SMD:R_0603_1608Metric_Pad0.98x0.95mm_HandSolder, F.Cu at (157.9, -10.7)
- added R8: 10k 1%, Resistor_SMD:R_0603_1608Metric_Pad0.98x0.95mm_HandSolder, F.Cu at (129.4, -8.16)
- added SW1: RST, Button_Switch_THT:SW_PUSH_6mm_H5mm, F.Cu at (222.0, -58.3)
- added SW2: SW_SPDT, Button_Switch_THT:SW_Slide_1P2T_CK_OS102011MS2Q, F.Cu at (154.5, 129.5)
- added U10: AT30TS75A-XM8M-T, Package_SO:MSOP-8_3x3mm_P0.65mm, F.Cu at (115.1, 9.07)
- added U11: M24256-BR (MB85RC16V), Package_SO:SOIC-8_3.9x4.9mm_P1.27mm, F.Cu at (107.2, 10.0)
- added U12: AMS1117-3.3, Package_TO_SOT_SMD:SOT-223-3_TabPin2, F.Cu at (119.8, -2.76)
- moved MCU1 22.9 mm to (158.8, 81.2)

Commit message: working on the charger
Parts:
- moved MCU1 8.75 mm to (167.5, 81.5), turned to -135 degrees

Commit message: Schematic in progress
Parts:
- added C10: 10u 10V, Capacitor_SMD:C_0805_2012Metric, F.Cu at (135.5, -69.0)
- added C11: 100n 50V, Capacitor_SMD:C_0603_1608Metric, F.Cu at (132.4, -57.7)
- added C12: 1u 10V, Capacitor_SMD:C_0603_1608Metric_Pad1.08x0.95mm_HandSolder, F.Cu at (122.8, -48.7)
- added C13: 100n 50V, Capacitor_SMD:C_0603_1608Metric, F.Cu at (127.0, -51.2)
- added C9: 100n 50V, Capacitor_SMD:C_0603_1608Metric, F.Cu at (141.5, -66.8)
- added D10: 30V 5A, Diode_SMD:D_SOD-128, F.Cu at (121.5, -63.9)
- added D11: 5.1V, Diode_SMD:D_SMA, F.Cu at (121.9, -68.2)
- added D12: ESDA6V1BC6, Package_TO_SOT_SMD:SOT-23-6, F.Cu at (114.0, -54.7)
- added D5: TVS, Diode_SMD:D_SMA, F.Cu at (110.3, -59.2)
- added D6: LED G, LED_SMD:LED_0603_1608Metric_Pad1.05x0.95mm_HandSolder, F.Cu at (109.7, -45.6)
- added D7: 30V 5A, Diode_SMD:D_SOD-128, F.Cu at (97.8, -44.1)
- added D8: 30V 5A, Diode_SMD:D_SOD-128, F.Cu at (129.6, -68.5)
- added D9: 30V 5A, Diode_SMD:D_SOD-128, F.Cu at (118.0, -59.4)
- added F3: 5A SLOW, Fuse:Fuse_1206_3216Metric_Pad1.42x1.75mm_HandSolder, F.Cu at (104.5, -44.5)
- added J3: CHG_IN, TerminalBlock:TerminalBlock_bornier-2_P5.08mm, F.Cu at (109.5, -66.0)
- added Q4: 2N7002NXAK, Package_TO_SOT_SMD:SOT-23, F.Cu at (113.9, -50.2)
- added Q5: 2N7002NXAK, Package_TO_SOT_SMD:SOT-23, F.Cu at (119.0, -55.2)
- added Q6: FZT549, Package_TO_SOT_SMD:SOT-223-3_TabPin2, F.Cu at (99.1, -50.3)
- added Q7: NX3008PBK,215, Package_TO_SOT_SMD:SOT-23, F.Cu at (128.3, -64.2)
- added Q8: PMOS, Package_TO_SOT_SMD:TO-252-2, F.Cu at (100.2, -66.5)
- added Q9: PMOS, Package_TO_SOT_SMD:TO-252-2, F.Cu at (100.2, -58.4)
- added R10: 100R 1%, Resistor_SMD:R_0603_1608Metric_Pad0.98x0.95mm_HandSolder, F.Cu at (139.9, -69.3)
- added R11: 10k 1%, Resistor_SMD:R_0603_1608Metric_Pad0.98x0.95mm_HandSolder, F.Cu at (118.4, -43.7)
- added R12: 10k 1%, Resistor_SMD:R_0603_1608Metric_Pad0.98x0.95mm_HandSolder, F.Cu at (137.3, -66.2)
- added R13: 150m, Resistor_SMD:R_0805_2012Metric_Pad1.20x1.40mm_HandSolder, F.Cu at (106.4, -48.4)
- added R14: 100R 1%, Resistor_SMD:R_0603_1608Metric_Pad0.98x0.95mm_HandSolder, F.Cu at (133.0, -65.2)
- added R15: 100k 1%, Resistor_SMD:R_0603_1608Metric_Pad0.98x0.95mm_HandSolder, F.Cu at (118.4, -46.2)
- added R16: 100R 1%, Resistor_SMD:R_0603_1608Metric_Pad0.98x0.95mm_HandSolder, F.Cu at (114.0, -46.8)
- added R17: 100R 1%, Resistor_SMD:R_0603_1608Metric_Pad0.98x0.95mm_HandSolder, F.Cu at (133.4, -60.2)
- added R18: 10k 1%, Resistor_SMD:R_0603_1608Metric_Pad0.98x0.95mm_HandSolder, F.Cu at (118.5, -48.7)
- added R19: 10k 1%, Resistor_SMD:R_0603_1608Metric_Pad0.98x0.95mm_HandSolder, F.Cu at (128.2, -56.2)
- added R20: 100k 1%, Resistor_SMD:R_0603_1608Metric_Pad0.98x0.95mm_HandSolder, F.Cu at (122.8, -51.2)
- added R21: 100k 1%, Resistor_SMD:R_0603_1608Metric_Pad0.98x0.95mm_HandSolder, F.Cu at (123.6, -53.7)
- added R22: 5k1 1%, Resistor_SMD:R_0603_1608Metric_Pad0.98x0.95mm_HandSolder, F.Cu at (118.5, -51.2)
- added R23: 5k1 1%, Resistor_SMD:R_0603_1608Metric_Pad0.98x0.95mm_HandSolder, F.Cu at (133.4, -62.7)
- added R24: 0R, Resistor_SMD:R_0603_1608Metric_Pad0.98x0.95mm_HandSolder, F.Cu at (114.0, -44.2)
- added R25: 0R, Resistor_SMD:R_0603_1608Metric_Pad0.98x0.95mm_HandSolder, F.Cu at (128.0, -53.7)
- added R26: 1k5 5%, Resistor_SMD:R_0603_1608Metric_Pad0.98x0.95mm_HandSolder, F.Cu at (123.9, -56.2)
- added R9: 10k 1%, Resistor_SMD:R_0603_1608Metric_Pad0.98x0.95mm_HandSolder, F.Cu at (129.0, -60.8)
- added U13: ADP2291, Package_SO:MSOP-8_3x3mm_P0.65mm, F.Cu at (107.7, -52.1)
- added U14: MCP6006R, Package_TO_SOT_SMD:SOT-23-5, F.Cu at (124.3, -59.7)
- D1: value TVS -> LED_ABGR; footprint Diode_SMD:D_SMA -> LED_SMD:LED_RGB_Wuerth-PLCC4_3.2x2.8mm_150141M173100
- D2: value TVS -> 5.1V
- J2: value BATTERY_OUT -> POWER_OUT
- MCU1: value STM32F407VETx -> STM32F407VGT6
- SW2: value SW_SPDT -> OS102011MS2QN1
- moved D1 8.40 mm to (132.2, -21.0)
Connections:
- C5 pad 1: +BATT -> +VDC
- C6 pad 1: +BATT -> +VDC
- D1 pad 1: Net-(D1-Pad1) -> unconnected-(D1-Pad1)
- D1 pad 2: GND -> unconnected-(D1-Pad2)
- D3 pad 1: unconnected-(D3-Pad1) -> Net-(D3-Pad1)
- D3 pad 2: unconnected-(D3-Pad2) -> GND
- F1 pad 2: Net-(D1-Pad1) -> Net-(F1-Pad2)
- F2 pad 2: Net-(D2-Pad1) -> Net-(F2-Pad2)
- J1 pad 1: unconnected-(J1-Pad1) -> Net-(J1-Pad1)
- J1 pad 2: unconnected-(J1-Pad2) -> GND
- J2 pad 1: +BATT -> +VDC
- Q1 pad 2: Net-(D1-Pad1) -> Net-(F1-Pad2)
- Q2 pad 2: Net-(D2-Pad1) -> Net-(F2-Pad2)
- Q3 pad 2: +BATT -> Net-(Q3-Pad2)
- R2 pad 1: Net-(D1-Pad1) -> Net-(F1-Pad2)
- R3 pad 1: Net-(D2-Pad1) -> Net-(F2-Pad2)
- R8 pad 2: +BATT -> +VDC
- SW2 pad 2: Net-(R7-Pad2) -> Net-(SW2-Pad2)
- SW2 pad 3: Net-(R7-Pad2) -> Net-(SW2-Pad2)
- U12 pad 3: +BATT -> +VDC

Commit message: schematic almost done
Parts:
- added C14: 100n 50V, Capacitor_SMD:C_0603_1608Metric, F.Cu at (3.50, -55.5)
- added C15: 100n 50V, Capacitor_SMD:C_0603_1608Metric, F.Cu at (1.70, -53.0)
- added C16: 20p 10V, Capacitor_SMD:C_0603_1608Metric_Pad1.08x0.95mm_HandSolder, F.Cu at (73.4, -79.6)
- added C17: 20p 10V, Capacitor_SMD:C_0603_1608Metric_Pad1.08x0.95mm_HandSolder, F.Cu at (73.4, -77.1)
- added C18: 2u2 6.3V, Capacitor_SMD:C_0603_1608Metric_Pad1.08x0.95mm_HandSolder, F.Cu at (73.4, -74.6)
- added C19: 2u2 6.3V, Capacitor_SMD:C_0603_1608Metric_Pad1.08x0.95mm_HandSolder, F.Cu at (77.8, -77.1)
- added C20: 100n 50V, Capacitor_SMD:C_0603_1608Metric, F.Cu at (77.6, -74.6)
- added C21: 100n 50V, Capacitor_SMD:C_0603_1608Metric, F.Cu at (73.2, -72.0)
- added C22: 16p 10V, Capacitor_SMD:C_0603_1608Metric_Pad1.08x0.95mm_HandSolder, F.Cu at (82.1, -79.6)
- added C23: 16p 10V, Capacitor_SMD:C_0603_1608Metric_Pad1.08x0.95mm_HandSolder, F.Cu at (77.8, -79.6)
- added C24: 100n 50V, Capacitor_SMD:C_0603_1608Metric, F.Cu at (78.7, -95.4)
- added C25: 100n 50V, Capacitor_SMD:C_0603_1608Metric, F.Cu at (90.5, -107.7)
- added C26: 100n 50V, Capacitor_SMD:C_0603_1608Metric, F.Cu at (73.2, -89.4)
- added C27: 100n 50V, Capacitor_SMD:C_0603_1608Metric, F.Cu at (86.8, -102.2)
- added C28: 100n 50V, Capacitor_SMD:C_0603_1608Metric, F.Cu at (95.2, -111.2)
- added C29: 100n 50V, Capacitor_SMD:C_0603_1608Metric, F.Cu at (83.1, -98.3)
- added C30: 100n 50V, Capacitor_SMD:C_0603_1608Metric, F.Cu at (44.2, -98.3)
- added C31: 1u 50V, Capacitor_SMD:C_0603_1608Metric, F.Cu at (37.9, -92.4)
- added C32: 10u 25V, Capacitor_SMD:C_0805_2012Metric, F.Cu at (29.1, -90.1)
- added C33: 1u 50V, Capacitor_SMD:C_0603_1608Metric, F.Cu at (37.7, -89.9)
- added C34: 10u 25V, Capacitor_SMD:C_0805_2012Metric, F.Cu at (33.7, -94.7)
- added C35: 1u 50V, Capacitor_SMD:C_0603_1608Metric, F.Cu at (48.4, -100.4)
- added C36: 100n 50V, Capacitor_SMD:C_0603_1608Metric, F.Cu at (52.6, -104.0)
- added C37: 100n 50V, Capacitor_SMD:C_0603_1608Metric, F.Cu at (61.8, -110.6)
- added C38: 100n 50V, Capacitor_SMD:C_0603_1608Metric, F.Cu at (60.7, -113.1)
- added C39: 100n 50V, Capacitor_SMD:C_0603_1608Metric_Pad1.08x0.95mm_HandSolder, F.Cu at (44.4, -104.4)
- added C40: 22u 16V, Capacitor_SMD:C_1206_3216Metric, F.Cu at (51.8, -79.2)
- added C41: 100n 50V, Capacitor_SMD:C_0603_1608Metric, F.Cu at (39.1, -57.2)
- added C42: 100n 50V, Capacitor_SMD:C_0603_1608Metric, F.Cu at (34.7, -50.0)
- added C43: 220p 50V, Capacitor_SMD:C_0603_1608Metric, F.Cu at (43.1, -57.2)
- added C44: 1u 50V, Capacitor_SMD:C_0603_1608Metric, F.Cu at (41.7, -59.7)
- added C45: 100n 50V, Capacitor_SMD:C_0603_1608Metric, F.Cu at (60.2, -76.2)
- added C46: 100n 50V, Capacitor_SMD:C_0603_1608Metric, F.Cu at (52.6, -68.0)
- added C47: 1u 50V, Capacitor_SMD:C_0603_1608Metric, F.Cu at (39.1, -54.7)
- added C48: 220p 50V, Capacitor_SMD:C_0603_1608Metric, F.Cu at (60.1, -73.7)
- added C49: 100n 50V, Capacitor_SMD:C_0603_1608Metric, F.Cu at (46.0, -60.4)
- added C50: 100n 50V, Capacitor_SMD:C_0603_1608Metric, F.Cu at (46.0, -63.0)
- added C51: 22u 16V, Capacitor_SMD:C_1206_3216Metric, F.Cu at (57.4, -79.2)
- added C52: 100n 50V, Capacitor_SMD:C_0603_1608Metric, F.Cu at (18.0, -72.8)
- added C53: 100n 50V, Capacitor_SMD:C_0603_1608Metric, F.Cu at (181.5, -78.5)
- added C54: 100n 50V, Capacitor_SMD:C_0603_1608Metric, F.Cu at (186.4, -88.2)
- added C55: 100n 50V, Capacitor_SMD:C_0603_1608Metric, F.Cu at (190.5, -88.2)
- added C56: 100n 50V, Capacitor_SMD:C_0603_1608Metric, F.Cu at (186.4, -85.7)
- added C57: 100n 50V, Capacitor_SMD:C_0603_1608Metric, F.Cu at (177.2, -76.0)
- added C58: 100n 50V, Capacitor_SMD:C_0603_1608Metric, F.Cu at (186.4, -83.2)
- added C59: 100n 50V, Capacitor_SMD:C_0603_1608Metric, F.Cu at (190.9, -91.2)
- added C60: 4.7u 10V, Capacitor_SMD:C_0805_2012Metric, F.Cu at (186.7, -91.0)
- added C61: 4.7u 10V, Capacitor_SMD:C_0805_2012Metric, F.Cu at (181.8, -81.3)
- added C62: 4.7u 10V, Capacitor_SMD:C_0805_2012Metric, F.Cu at (177.4, -81.3)
- added C63: 1u 10V, Capacitor_SMD:C_0603_1608Metric_Pad1.08x0.95mm_HandSolder, F.Cu at (177.3, -78.5)
- added D13: RGB_LED, LED_SMD:LED_RGB_Wuerth-PLCC4_3.2x2.8mm_150141M173100, F.Cu at (-19.2, -67.5)
- added D14: RGB_LED, LED_SMD:LED_RGB_Wuerth-PLCC4_3.2x2.8mm_150141M173100, F.Cu at (-6.91, -71.8)
- added D15: RGB_LED, LED_SMD:LED_RGB_Wuerth-PLCC4_3.2x2.8mm_150141M173100, F.Cu at (-24.1, -56.7)
- added D16: RGB_LED, LED_SMD:LED_RGB_Wuerth-PLCC4_3.2x2.8mm_150141M173100, F.Cu at (-13.1, -71.8)
- added D17: RGB_LED, LED_SMD:LED_RGB_Wuerth-PLCC4_3.2x2.8mm_150141M173100, F.Cu at (-30.3, -48.0)
- added D18: RGB_LED, LED_SMD:LED_RGB_Wuerth-PLCC4_3.2x2.8mm_150141M173100, F.Cu at (-19.2, -63.1)
- added D19: RGB_LED, LED_SMD:LED_RGB_Wuerth-PLCC4_3.2x2.8mm_150141M173100, F.Cu at (-30.3, -52.3)
- added D20: RGB_LED, LED_SMD:LED_RGB_Wuerth-PLCC4_3.2x2.8mm_150141M173100, F.Cu at (-30.3, -56.7)
- added D21: RGB_LED, LED_SMD:LED_RGB_Wuerth-PLCC4_3.2x2.8mm_150141M173100, F.Cu at (-19.2, -71.8)
- added D22: RGB_LED, LED_SMD:LED_RGB_Wuerth-PLCC4_3.2x2.8mm_150141M173100, F.Cu at (-13.1, -67.5)
- added D23: 30V 5A, Diode_SMD:D_SOD-128, F.Cu at (47.8, -115.9)
- added D24: LED G, LED_SMD:LED_0603_1608Metric_Pad1.05x0.95mm_HandSolder, F.Cu at (228.2, -91.2)
- added J10: I2C_MONITOR, Connector_PinHeader_2.54mm:PinHeader_2x02_P2.54mm_Vertical, F.Cu at (46.5, -111.6)
- added J11: EXT_MODULE, Connector_IDC:IDC-Header_2x10_P2.54mm_Vertical, F.Cu at (-28.1, -111.8)
- added J12: MINI_MOD_A, Connector_IDC:IDC-Header_2x05_P2.54mm_Vertical, F.Cu at (-4.13, -111.8)
- added J13: MINI_MOD_B, Connector_IDC:IDC-Header_2x05_P2.54mm_Vertical, F.Cu at (-16.1, -111.8)
- added J14: AUX_PROG, Connector_PinHeader_2.54mm:PinHeader_1x06_P2.54mm_Vertical, F.Cu at (-16.5, -93.2)
- added J15: Motor_L, Connector_PinHeader_2.54mm:PinHeader_1x06_P2.54mm_Vertical, F.Cu at (39.7, -78.5)
- added J16: Motor_R, Connector_PinHeader_2.54mm:PinHeader_1x06_P2.54mm_Vertical, F.Cu at (35.0, -78.5)
- added J17: UART_Bridge, Connector_PinHeader_2.54mm:PinHeader_1x03_P2.54mm_Vertical, F.Cu at (177.5, -90.1)
- added J18: I2C_Bridge, Connector_PinHeader_2.54mm:PinHeader_1x03_P2.54mm_Vertical, F.Cu at (182.1, -90.1)
- added J19: PMOD_I2C, Connector_PinSocket_2.54mm:PinSocket_2x04_P2.54mm_Vertical, F.Cu at (210.2, -90.1)
- added J5: BOOT_SEL, Connector_PinHeader_2.54mm:PinHeader_1x03_P2.54mm_Vertical, F.Cu at (68.9, -78.5)
- added J6: SONAR_MONITOR, Connector_PinHeader_2.54mm:PinHeader_2x02_P2.54mm_Vertical, F.Cu at (53.8, -115.6)
- added J7: Molex 104031-0811, Connector_Card:microSD_HC_Molex_104031-0811, F.Cu at (29.6, -107.7)
- added J8: HY-SRF05, Connector_PinSocket_2.54mm:PinSocket_1x05_P2.54mm_Vertical, F.Cu at (24.6, -98.3)
- added J9: ESP8266-01, Connector_PinSocket_2.54mm:PinSocket_2x04_P2.54mm_Vertical, F.Cu at (41.9, -115.6)
- added L1: 4.7uH, Inductor_SMD:L_Wuerth_MAPI-3020, F.Cu at (39.6, -103.2)
- added Q10: 2N7002NXAK, Package_TO_SOT_SMD:SOT-23, F.Cu at (-24.7, -52.3)
- added Q11: 2N7002NXAK, Package_TO_SOT_SMD:SOT-23, F.Cu at (-7.54, -67.4)
- added Q12: 2N7002NXAK, Package_TO_SOT_SMD:SOT-23, F.Cu at (-18.6, -58.7)
- added Q13: 2N7002NXAK, Package_TO_SOT_SMD:SOT-23, F.Cu at (-1.39, -71.8)
- added Q14: 2N7002NXAK, Package_TO_SOT_SMD:SOT-23, F.Cu at (-30.9, -43.6)
- added Q15: 2N7002NXAK, Package_TO_SOT_SMD:SOT-23, F.Cu at (-13.7, -63.1)
- added Q16: 2N7002NXAK, Package_TO_SOT_SMD:SOT-23, F.Cu at (34.5, -98.4)
- added Q17: 2N7002NXAK, Package_TO_SOT_SMD:SOT-23, F.Cu at (44.5, -74.0)
- added Q18: 2N7002NXAK, Package_TO_SOT_SMD:SOT-23, F.Cu at (51.4, -75.3)
- added R100: 4k7 1%, Resistor_SMD:R_0603_1608Metric, F.Cu at (48.6, -105.4)
- added R101: 10k 1%, Resistor_SMD:R_0603_1608Metric, F.Cu at (53.4, -106.5)
- added R102: 4k7 1%, Resistor_SMD:R_0603_1608Metric, F.Cu at (42.2, -92.4)
- added R103: 5k1 1%, Resistor_SMD:R_0603_1608Metric_Pad0.98x0.95mm_HandSolder, F.Cu at (38.1, -94.9)
- added R104: 10k 1%, Resistor_SMD:R_0603_1608Metric, F.Cu at (57.4, -106.5)
- added R105: 110k 1%, Resistor_SMD:R_0603_1608Metric, F.Cu at (33.2, -87.4)
- added R106: 15k 1%, Resistor_SMD:R_0603_1608Metric, F.Cu at (57.8, -109.5)
- added R107: 2k2 1%, Resistor_SMD:R_0603_1608Metric, F.Cu at (48.2, -97.9)
- added R108: 2k2 1%, Resistor_SMD:R_0603_1608Metric, F.Cu at (37.2, -87.4)
- added R109: 100R 1%, Resistor_SMD:R_0603_1608Metric_Pad0.98x0.95mm_HandSolder, F.Cu at (41.8, -62.2)
- added R110: 10k 1%, Resistor_SMD:R_0603_1608Metric_Pad0.98x0.95mm_HandSolder, F.Cu at (34.9, -55.1)
- added R111: 10k 1%, Resistor_SMD:R_0603_1608Metric_Pad0.98x0.95mm_HandSolder, F.Cu at (44.2, -70.5)
- added R112: 0R 5%, Resistor_SMD:R_0603_1608Metric_Pad0.98x0.95mm_HandSolder, F.Cu at (48.5, -70.5)
- added R113: 0R 5% (DNP), Resistor_SMD:R_0603_1608Metric_Pad0.98x0.95mm_HandSolder, F.Cu at (44.2, -68.0)
- added R114: 10k 1%, Resistor_SMD:R_0603_1608Metric_Pad0.98x0.95mm_HandSolder, F.Cu at (34.9, -52.6)
- added R115: 100R 1%, Resistor_SMD:R_0603_1608Metric_Pad0.98x0.95mm_HandSolder, F.Cu at (44.2, -65.5)
- added R116: 0R 5%, Resistor_SMD:R_0603_1608Metric_Pad0.98x0.95mm_HandSolder, F.Cu at (56.0, -76.2)
- added R117: 0R 5% (DNP), Resistor_SMD:R_0603_1608Metric_Pad0.98x0.95mm_HandSolder, F.Cu at (34.9, -57.6)
- added R118: 2k2 1%, Resistor_SMD:R_0603_1608Metric, F.Cu at (162.6, -51.5)
- added R119: 2k2 1%, Resistor_SMD:R_0603_1608Metric, F.Cu at (158.6, -51.5)
- added R120: 10k 1%, Resistor_SMD:R_0603_1608Metric_Pad0.98x0.95mm_HandSolder, F.Cu at (228.1, -88.6)
- added R27: 330R 5%, Resistor_SMD:R_0805_2012Metric, F.Cu at (-11.3, -51.9)
- added R28: 330R 5%, Resistor_SMD:R_0805_2012Metric, F.Cu at (-9.04, -63.7)
- added R29: 330R 5%, Resistor_SMD:R_0805_2012Metric, F.Cu at (-9.53, -57.8)
- added R30: 330R 5%, Resistor_SMD:R_0805_2012Metric, F.Cu at (-18.8, -55.0)
- added R31: 330R 5%, Resistor_SMD:R_0805_2012Metric, F.Cu at (-25.0, -45.6)
- added R32: 330R 5%, Resistor_SMD:R_0805_2012Metric, F.Cu at (-11.8, -49.0)
- added R33: 330R 5%, Resistor_SMD:R_0805_2012Metric, F.Cu at (-4.63, -63.7)
- added R34: 330R 5%, Resistor_SMD:R_0805_2012Metric, F.Cu at (-20.1, -52.1)
- added R35: 330R 5%, Resistor_SMD:R_0805_2012Metric, F.Cu at (-2.89, -68.1)
- added R36: 330R 5%, Resistor_SMD:R_0805_2012Metric, F.Cu at (4.19, -63.7)
- added R37: 330R 5%, Resistor_SMD:R_0805_2012Metric, F.Cu at (-9.53, -54.9)
- added R38: 330R 5%, Resistor_SMD:R_0805_2012Metric, F.Cu at (-11.8, -46.0)
- added R39: 330R 5%, Resistor_SMD:R_0805_2012Metric, F.Cu at (-5.12, -57.8)
- added R40: 330R 5%, Resistor_SMD:R_0805_2012Metric, F.Cu at (-26.2, -42.7)
- added R41: 330R 5%, Resistor_SMD:R_0805_2012Metric, F.Cu at (5.93, -69.6)
- added R42: 330R 5%, Resistor_SMD:R_0805_2012Metric, F.Cu at (-5.12, -54.9)
- added R43: 330R 5%, Resistor_SMD:R_0805_2012Metric, F.Cu at (5.93, -66.6)
- added R44: 330R 5%, Resistor_SMD:R_0805_2012Metric, F.Cu at (-21.8, -42.7)
- added R45: 330R 5%, Resistor_SMD:R_0805_2012Metric, F.Cu at (-13.9, -59.4)
- added R46: 330R 5%, Resistor_SMD:R_0805_2012Metric, F.Cu at (4.19, -60.7)
- added R47: 330R 5%, Resistor_SMD:R_0805_2012Metric, F.Cu at (3.26, -72.5)
- added R48: 330R 5%, Resistor_SMD:R_0805_2012Metric, F.Cu at (-16.2, -49.1)
- added R49: 330R 5%, Resistor_SMD:R_0805_2012Metric, F.Cu at (-20.6, -48.6)
- added R50: 330R 5%, Resistor_SMD:R_0805_2012Metric, F.Cu at (-15.7, -52.1)
- added R51: 330R 5%, Resistor_SMD:R_0805_2012Metric, F.Cu at (7.67, -72.5)
- added R52: 330R 5%, Resistor_SMD:R_0805_2012Metric, F.Cu at (-7.34, -49.0)
- added R53: 330R 5%, Resistor_SMD:R_0805_2012Metric, F.Cu at (-13.9, -56.4)
- added R54: 330R 5%, Resistor_SMD:R_0805_2012Metric, F.Cu at (-16.2, -46.2)
- added R55: 330R 5%, Resistor_SMD:R_0805_2012Metric, F.Cu at (-0.22, -62.2)
- added R56: 330R 5%, Resistor_SMD:R_0805_2012Metric, F.Cu at (-4.63, -60.8)
- added R57: 100R 1%, Resistor_SMD:R_0805_2012Metric, F.Cu at (-20.6, -45.6)
- added R58: 100R 1%, Resistor_SMD:R_0805_2012Metric, F.Cu at (-0.22, -65.1)
- added R59: 100R 1%, Resistor_SMD:R_0805_2012Metric, F.Cu at (-9.04, -60.8)
- added R60: 10k 1%, Resistor_SMD:R_0603_1608Metric_Pad0.98x0.95mm_HandSolder, F.Cu at (4.16, -58.0)
- added R61: 10k 1%, Resistor_SMD:R_0603_1608Metric_Pad0.98x0.95mm_HandSolder, F.Cu at (-8.69, -43.3)
- added R62: 10k 1%, Resistor_SMD:R_0603_1608Metric_Pad0.98x0.95mm_HandSolder, F.Cu at (8.57, -63.9)
- added R63: 100R 1%, Resistor_SMD:R_0805_2012Metric, F.Cu at (-0.22, -59.2)
- added R64: 10k 1%, Resistor_SMD:R_0603_1608Metric_Pad0.98x0.95mm_HandSolder, F.Cu at (-2.96, -49.2)
- added R65: 100R 1%, Resistor_SMD:R_0805_2012Metric, F.Cu at (-0.71, -56.3)
- added R66: 10k 1%, Resistor_SMD:R_0603_1608Metric_Pad0.98x0.95mm_HandSolder, F.Cu at (-2.48, -52.2)
- added R67: 330R 5%, Resistor_SMD:R_0805_2012Metric, F.Cu at (-17.4, -42.7)
- added R68: 330R 5%, Resistor_SMD:R_0805_2012Metric, F.Cu at (10.3, -66.6)
- added R69: 330R 5%, Resistor_SMD:R_0805_2012Metric, F.Cu at (-6.86, -51.9)
- added R70: 100R 1%, Resistor_SMD:R_0805_2012Metric, F.Cu at (-25.0, -48.6)
- added R71: 10k 1%, Resistor_SMD:R_0603_1608Metric_Pad0.98x0.95mm_HandSolder, F.Cu at (8.57, -61.4)
- added R72: 10k 1%, Resistor_SMD:R_0603_1608Metric_Pad0.98x0.95mm_HandSolder, F.Cu at (-7.37, -46.3)
- added R73: 10k 1%, Resistor_SMD:R_0603_1608Metric_Pad0.98x0.95mm_HandSolder, F.Cu at (-13.0, -43.3)
- added R74: 100R 1%, Resistor_SMD:R_0805_2012Metric, F.Cu at (1.52, -68.1)
- added R75: 100R 1%, Resistor_SMD:R_0805_2012Metric, F.Cu at (10.3, -69.6)
- added R76: 10k 1%, Resistor_SMD:R_0603_1608Metric_Pad0.98x0.95mm_HandSolder, F.Cu at (69.0, -89.9)
- added R77: 147R 1%, Resistor_SMD:R_0805_2012Metric_Pad1.20x1.40mm_HandSolder, F.Cu at (86.1, -107.5)
- added R78: 3k3 1%, Resistor_SMD:R_0603_1608Metric_Pad0.98x0.95mm_HandSolder, F.Cu at (74.1, -94.4)
- added R79: 147R 1%, Resistor_SMD:R_0805_2012Metric_Pad1.20x1.40mm_HandSolder, F.Cu at (90.8, -110.4)
- added R80: 3k3 1%, Resistor_SMD:R_0603_1608Metric_Pad0.98x0.95mm_HandSolder, F.Cu at (97.0, -114.2)
- added R81: 147R 1%, Resistor_SMD:R_0805_2012Metric_Pad1.20x1.40mm_HandSolder, F.Cu at (92.4, -116.5)
- added R82: 3k3 1%, Resistor_SMD:R_0603_1608Metric_Pad0.98x0.95mm_HandSolder, F.Cu at (86.9, -104.7)
- added R83: 147R 1%, Resistor_SMD:R_0805_2012Metric_Pad1.20x1.40mm_HandSolder, F.Cu at (82.4, -103.6)
- added R84: 3k3 1%, Resistor_SMD:R_0603_1608Metric_Pad0.98x0.95mm_HandSolder, F.Cu at (82.2, -100.8)
- added R85: 147R 1%, Resistor_SMD:R_0805_2012Metric_Pad1.20x1.40mm_HandSolder, F.Cu at (86.1, -110.4)
- added R86: 3k3 1%, Resistor_SMD:R_0603_1608Metric_Pad0.98x0.95mm_HandSolder, F.Cu at (97.0, -116.7)
- added R87: 147R 1%, Resistor_SMD:R_0805_2012Metric_Pad1.20x1.40mm_HandSolder, F.Cu at (74.3, -97.1)
- added R88: 3k3 1%, Resistor_SMD:R_0603_1608Metric_Pad0.98x0.95mm_HandSolder, F.Cu at (73.7, -91.9)
- added R89: 147R 1%, Resistor_SMD:R_0805_2012Metric_Pad1.20x1.40mm_HandSolder, F.Cu at (77.6, -100.6)
- added R90: 3k3 1%, Resistor_SMD:R_0603_1608Metric_Pad0.98x0.95mm_HandSolder, F.Cu at (69.0, -87.4)
- added R91: 147R 1%, Resistor_SMD:R_0805_2012Metric_Pad1.20x1.40mm_HandSolder, F.Cu at (69.2, -92.7)
- added R92: 3k3 1%, Resistor_SMD:R_0603_1608Metric_Pad0.98x0.95mm_HandSolder, F.Cu at (78.9, -97.9)
- added R93: 147R 1%, Resistor_SMD:R_0805_2012Metric_Pad1.20x1.40mm_HandSolder, F.Cu at (77.6, -103.6)
- added R94: 3k3 1%, Resistor_SMD:R_0603_1608Metric_Pad0.98x0.95mm_HandSolder, F.Cu at (92.2, -113.7)
- added R95: 10R 1%, Resistor_SMD:R_0805_2012Metric, F.Cu at (53.6, -109.3)
- added R96: 10k 1%, Resistor_SMD:R_0603_1608Metric_Pad0.98x0.95mm_HandSolder, F.Cu at (33.5, -90.4)
- added R97: 4k7 1%, Resistor_SMD:R_0603_1608Metric, F.Cu at (42.2, -94.9)
- added R98: 4k7 1%, Resistor_SMD:R_0603_1608Metric, F.Cu at (48.6, -102.9)
- added R99: 4k7 1%, Resistor_SMD:R_0603_1608Metric_Pad0.98x0.95mm_HandSolder, F.Cu at (29.1, -87.4)
- added RV1: 100k POT, Potentiometer_SMD:Potentiometer_Bourns_3224W_Vertical, F.Cu at (86.9, -114.9)
- added SW3: BTN, Button_Switch_SMD:SW_Push_1P1T_NO_6x6mm_H9.5mm, F.Cu at (-27.8, -62.6)
- added SW4: BTN, Button_Switch_SMD:SW_Push_1P1T_NO_6x6mm_H9.5mm, F.Cu at (-27.8, -70.2)
- added TP1: TestPoint, TestPoint:TestPoint_THTPad_D2.5mm_Drill1.2mm, F.Cu at (29.2, -93.9)
- added TP2: TestPoint, TestPoint:TestPoint_THTPad_D2.5mm_Drill1.2mm, F.Cu at (158.8, -58.6)
- added U15: AP2171AW-7, Package_TO_SOT_SMD:SOT-23-5, F.Cu at (69.4, -96.4)
- added U16: LM393, Package_SO:SOIC-8_3.9x4.9mm_P1.27mm, F.Cu at (79.5, -108.3)
- added U17: LM393, Package_SO:SOIC-8_3.9x4.9mm_P1.27mm, F.Cu at (71.0, -108.3)
- added U18: LM393, Package_SO:SOIC-8_3.9x4.9mm_P1.27mm, F.Cu at (71.0, -101.8)
- added U19: LM393, Package_SO:SOIC-8_3.9x4.9mm_P1.27mm, F.Cu at (71.0, -114.7)
- added U20: LM393, Package_SO:SOIC-8_3.9x4.9mm_P1.27mm, F.Cu at (79.5, -114.7)
- added U21: SN74LVC1G14DBV, Package_TO_SOT_SMD:SOT-23-5, F.Cu at (29.5, -98.4)
- added U22: MT3608, Package_TO_SOT_SMD:SOT-23-6, F.Cu at (39.6, -98.4)
- added U23: APDS-9306-065, OptoDevice:Broadcom_DFN-6_2x2mm_P0.65mm, F.Cu at (60.9, -116.2)
- added U24: SHTC3, Sensor_Humidity:Sensirion_DFN-4-1EP_2x2mm_P1mm_EP0.7x1.6mm, F.Cu at (52.6, -101.0)
- added U25: DPS310XTSA1, Package_LGA:Bosch_LGA-8_2x2.5mm_P0.65mm_ClockwisePinNumbering, F.Cu at (44.3, -101.4)
- added U26: MC6470, Package_LGA:LGA-12_2x2mm_P0.5mm, F.Cu at (46.0, -94.9)
- added U27: DRV8212DSG, Package_SON:WSON-8-1EP_2x2mm_P0.5mm_EP0.9x1.6mm_ThermalVias, F.Cu at (48.5, -67.5)
- added U28: 74HC2G08DP,125, Package_SO:TSSOP-8_3x3mm_P0.65mm, F.Cu at (36.2, -61.2)
- added U29: 74HC2G08DP,125, Package_SO:TSSOP-8_3x3mm_P0.65mm, F.Cu at (45.5, -78.5)
- added U30: DRV8212DSG, Package_SON:WSON-8-1EP_2x2mm_P0.5mm_EP0.9x1.6mm_ThermalVias, F.Cu at (56.0, -73.2)
- added U31: STLINK_V3MODS, STLINK_V3MODS:STLINK-V3MODS, F.Cu at (165.7, -74.1)
- D1: value LED_ABGR -> RGB_LED
- U12: value AMS1117-3.3 -> TC1108-3.3
Connections:
- net /Power/BJ_BUS renamed /BARREL_JACK_BUS
- D1 pad 1: unconnected-(D1-Pad1) -> +VDC
- D1 pad 2: unconnected-(D1-Pad2) -> Net-(D1-Pad2)
- D1 pad 3: unconnected-(D1-Pad3) -> Net-(D1-Pad3)
- D1 pad 4: unconnected-(D1-Pad4) -> Net-(D1-Pad4)
- MCU1 pad 1: unconnected-(MCU1-Pad1) -> /ESP_CH_PD/EN
- MCU1 pad 10: unconnected-(MCU1-Pad10) -> GND
- MCU1 pad 100: unconnected-(MCU1-Pad100) -> +3V3
- MCU1 pad 11: unconnected-(MCU1-Pad11) -> +3V3
- MCU1 pad 12: unconnected-(MCU1-Pad12) -> Net-(MCU1-Pad12)
- MCU1 pad 13: unconnected-(MCU1-Pad13) -> Net-(MCU1-Pad13)
- MCU1 pad 14: unconnected-(MCU1-Pad14) -> /MCU/NRST
- MCU1 pad 15: unconnected-(MCU1-Pad15) -> /MINI_B_0
- MCU1 pad 16: unconnected-(MCU1-Pad16) -> /MINI_B_1
- MCU1 pad 17: unconnected-(MCU1-Pad17) -> /EXT1
- MCU1 pad 18: unconnected-(MCU1-Pad18) -> /EXT2
- MCU1 pad 19: unconnected-(MCU1-Pad19) -> +3V3
- MCU1 pad 2: unconnected-(MCU1-Pad2) -> /ESP_GPIO2
- MCU1 pad 20: unconnected-(MCU1-Pad20) -> GND
- MCU1 pad 21: unconnected-(MCU1-Pad21) -> +3V3
- MCU1 pad 22: unconnected-(MCU1-Pad22) -> +3V3
- MCU1 pad 23: unconnected-(MCU1-Pad23) -> /EXT6
- MCU1 pad 24: unconnected-(MCU1-Pad24) -> /LED_USER_R
- MCU1 pad 25: unconnected-(MCU1-Pad25) -> /LED_USER_G
- MCU1 pad 26: unconnected-(MCU1-Pad26) -> /LED_USER_B
- MCU1 pad 27: unconnected-(MCU1-Pad27) -> GND
- MCU1 pad 28: unconnected-(MCU1-Pad28) -> +3V3
- MCU1 pad 29: unconnected-(MCU1-Pad29) -> /EXT7
- MCU1 pad 3: unconnected-(MCU1-Pad3) -> /ESP_GPIO0
- MCU1 pad 30: unconnected-(MCU1-Pad30) -> /SD_CLK
- MCU1 pad 31: unconnected-(MCU1-Pad31) -> /SD_DATA_OUT
- MCU1 pad 32: unconnected-(MCU1-Pad32) -> /SD_DATA_IN
- MCU1 pad 33: unconnected-(MCU1-Pad33) -> /VOLTAGE_MONITOR
- MCU1 pad 34: unconnected-(MCU1-Pad34) -> /MINI_A_2
- MCU1 pad 35: unconnected-(MCU1-Pad35) -> /EXT9
- MCU1 pad 36: unconnected-(MCU1-Pad36) -> /EXT10
- MCU1 pad 37: unconnected-(MCU1-Pad37) -> /EXT11
- MCU1 pad 38: unconnected-(MCU1-Pad38) -> /MINI_A_0
- MCU1 pad 39: unconnected-(MCU1-Pad39) -> /MINI_A_1
- MCU1 pad 4: unconnected-(MCU1-Pad4) -> /SONAR_ECHO
- MCU1 pad 40: unconnected-(MCU1-Pad40) -> /ENC_R_A
- MCU1 pad 41: unconnected-(MCU1-Pad41) -> /SONAR_ENA
- MCU1 pad 42: unconnected-(MCU1-Pad42) -> /ENC_R_B
- MCU1 pad 43: unconnected-(MCU1-Pad43) -> /SENSORS_ENABLE
- MCU1 pad 44: unconnected-(MCU1-Pad44) -> /LED_DECOR_R
- MCU1 pad 45: unconnected-(MCU1-Pad45) -> /LED_DECOR_G
- MCU1 pad 46: unconnected-(MCU1-Pad46) -> /LED_DECOR_B
- MCU1 pad 47: unconnected-(MCU1-Pad47) -> /MODULE_SCL
- MCU1 pad 48: unconnected-(MCU1-Pad48) -> /MODULE_SDA
- MCU1 pad 49: unconnected-(MCU1-Pad49) -> Net-(MCU1-Pad49)
- MCU1 pad 5: unconnected-(MCU1-Pad5) -> /ESP_RST
- MCU1 pad 50: unconnected-(MCU1-Pad50) -> +3V3
- MCU1 pad 51: unconnected-(MCU1-Pad51) -> /DEBUG_LED
- MCU1 pad 52: unconnected-(MCU1-Pad52) -> /EXT0
- MCU1 pad 53: unconnected-(MCU1-Pad53) -> /MINI_A_3
- MCU1 pad 54: unconnected-(MCU1-Pad54) -> /MINI_A_4
- MCU1 pad 55: unconnected-(MCU1-Pad55) -> /SENSOR_6
- MCU1 pad 56: unconnected-(MCU1-Pad56) -> /SENSOR_7
- MCU1 pad 57: unconnected-(MCU1-Pad57) -> /SENSOR_8
- MCU1 pad 58: unconnected-(MCU1-Pad58) -> /SENSOR_9
- MCU1 pad 59: unconnected-(MCU1-Pad59) -> /ENC_L_A
- MCU1 pad 6: unconnected-(MCU1-Pad6) -> +3V3
- MCU1 pad 60: unconnected-(MCU1-Pad60) -> /ENC_L_B
- MCU1 pad 61: unconnected-(MCU1-Pad61) -> /INT_ACC
- MCU1 pad 62: unconnected-(MCU1-Pad62) -> /INT_MAG
- MCU1 pad 63: unconnected-(MCU1-Pad63) -> /MOTOR_R_EN
- MCU1 pad 64: unconnected-(MCU1-Pad64) -> /MOTOR_R_PH
- MCU1 pad 65: unconnected-(MCU1-Pad65) -> /MOTOR_L_EN
- MCU1 pad 66: unconnected-(MCU1-Pad66) -> /MOTOR_L_PH
- MCU1 pad 67: unconnected-(MCU1-Pad67) -> /EXT8
- MCU1 pad 68: unconnected-(MCU1-Pad68) -> /ESP_RX
- MCU1 pad 69: unconnected-(MCU1-Pad69) -> /ESP_TX
- MCU1 pad 7: unconnected-(MCU1-Pad7) -> /EXT5
- MCU1 pad 70: unconnected-(MCU1-Pad70) -> /USB_DM
- MCU1 pad 71: unconnected-(MCU1-Pad71) -> /USB_DP
- MCU1 pad 72: unconnected-(MCU1-Pad72) -> /MCU/STLINK_SWDIO
- MCU1 pad 73: unconnected-(MCU1-Pad73) -> Net-(MCU1-Pad73)
- MCU1 pad 74: unconnected-(MCU1-Pad74) -> GND
- MCU1 pad 75: unconnected-(MCU1-Pad75) -> +3V3
- MCU1 pad 76: unconnected-(MCU1-Pad76) -> /MCU/STLINK_SWCLK
- MCU1 pad 77: unconnected-(MCU1-Pad77) -> /USB_DP_PULL
- MCU1 pad 78: unconnected-(MCU1-Pad78) -> /EXT3
- MCU1 pad 79: unconnected-(MCU1-Pad79) -> /EXT4
- MCU1 pad 8: unconnected-(MCU1-Pad8) -> Net-(MCU1-Pad8)
- MCU1 pad 80: unconnected-(MCU1-Pad80) -> /MCU/STLINK_VCP_RX
- MCU1 pad 81: unconnected-(MCU1-Pad81) -> /BUTTON_1
- MCU1 pad 82: unconnected-(MCU1-Pad82) -> /BUTTON_2
- MCU1 pad 83: unconnected-(MCU1-Pad83) -> /MCU/STLINK_VCP_TX
- MCU1 pad 84: unconnected-(MCU1-Pad84) -> /SENSOR_1
- MCU1 pad 85: unconnected-(MCU1-Pad85) -> /SENSOR_2
- MCU1 pad 86: unconnected-(MCU1-Pad86) -> /SENSOR_3
- MCU1 pad 87: unconnected-(MCU1-Pad87) -> /SENSOR_4
- MCU1 pad 88: unconnected-(MCU1-Pad88) -> /SENSOR_5
- MCU1 pad 89: unconnected-(MCU1-Pad89) -> /MCU/STLINK_SWO
- MCU1 pad 9: unconnected-(MCU1-Pad9) -> Net-(MCU1-Pad9)
- MCU1 pad 90: unconnected-(MCU1-Pad90) -> /MINI_B_2
- MCU1 pad 91: unconnected-(MCU1-Pad91) -> /MINI_B_3
- MCU1 pad 92: unconnected-(MCU1-Pad92) -> /PRH_SCL
- MCU1 pad 93: unconnected-(MCU1-Pad93) -> /PRH_SDA
- MCU1 pad 94: unconnected-(MCU1-Pad94) -> Net-(MCU1-Pad94)
- MCU1 pad 95: unconnected-(MCU1-Pad95) -> /SONAR_TRIG
- MCU1 pad 96: unconnected-(MCU1-Pad96) -> /MINI_B_4
- MCU1 pad 97: unconnected-(MCU1-Pad97) -> /SD_CS
- MCU1 pad 98: unconnected-(MCU1-Pad98) -> /SD_DETECT
- MCU1 pad 99: unconnected-(MCU1-Pad99) -> GND
- R24 pad 2: /Power/USB_DM -> /USB_DM
- R25 pad 2: /Power/USB_DP -> /USB_DP
- R26 pad 1: /Power/USB_DP -> /USB_DP
- R26 pad 2: /Power/USB_DP_PULL -> /USB_DP_PULL
- U1 pad 1: unconnected-(U1-Pad1) -> Net-(U1-Pad1)
- U1 pad 2: unconnected-(U1-Pad2) -> GND
- U1 pad 3: unconnected-(U1-Pad3) -> GND
- U1 pad 4: unconnected-(U1-Pad4) -> /line_sensors/S1
- U10 pad 1: /Peripherals/SDA -> /PRH_SDA
- U10 pad 2: /Peripherals/SCL -> /PRH_SCL
- U11 pad 5: /Peripherals/SDA -> /PRH_SDA
- U11 pad 6: /Peripherals/SCL -> /PRH_SCL
- U11 pad 7: /Peripherals/MEM_WC -> unconnected-(U11-Pad7)
- U12 pad 1: GND -> +VDC
- U12 pad 2: +3V3 -> GND
- U12 pad 3: +VDC -> +3V3
- U14 pad 1: /Power/VOLTAGE_MONITOR -> /VOLTAGE_MONITOR
- U14 pad 4: /Power/VOLTAGE_MONITOR -> /VOLTAGE_MONITOR
- U2 pad 1: unconnected-(U2-Pad1) -> Net-(U2-Pad1)
- U2 pad 2: unconnected-(U2-Pad2) -> GND
- U2 pad 3: unconnected-(U2-Pad3) -> GND
- U2 pad 4: unconnected-(U2-Pad4) -> /line_sensors/S2
- U3 pad 1: unconnected-(U3-Pad1) -> Net-(U3-Pad1)
- U3 pad 2: unconnected-(U3-Pad2) -> GND
- U3 pad 3: unconnected-(U3-Pad3) -> GND
- U3 pad 4: unconnected-(U3-Pad4) -> /line_sensors/S3
- U4 pad 1: unconnected-(U4-Pad1) -> Net-(U4-Pad1)
- U4 pad 2: unconnected-(U4-Pad2) -> GND
- U4 pad 3: unconnected-(U4-Pad3) -> GND
- U4 pad 4: unconnected-(U4-Pad4) -> /line_sensors/S4
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
Commit message: Layout in progress
Parts:
- C40, C41, C42, C43, C44, C47, C48, C49, C50, C51, D1, D13, D14, D15, D16, D17, D18, D19, D20, D21, R112, R113, R116, R117, U27, U30: moved to B.Cu
- H11, H12, H13, H14, H15: value Bumper_hole -> Bumber_hole
- SW1: footprint Button_Switch_THT:SW_PUSH_6mm_H5mm -> Button_Switch_SMD:SW_Push_1P1T_NO_6x6mm_H9.5mm
- moved D15 324.0 mm to (242.5, 127.5), turned to 90 degrees
- moved J14 288.8 mm to (189.1, 109.7), turned to 7 degrees
- moved U18 279.5 mm to (245.0, 117.0), turned to -90 degrees
- moved D16 277.5 mm to (185.0, 122.5), turned to 180 degrees
- moved J8 277.4 mm to (230.5, 87.6), turned to 180 degrees
- moved C27 273.9 mm to (248.6, 118.7), turned to 90 degrees
- moved D14 272.3 mm to (242.5, 37.5), turned to 90 degrees
- moved U17 269.8 mm to (245.0, 98.0), turned to -90 degrees
- moved J7 265.1 mm to (158.9, 123.8), turned to 7 degrees
- moved C26 257.9 mm to (248.6, 99.7), turned to 90 degrees
- moved U16 252.6 mm to (245.0, 82.5), turned to -90 degrees
- moved U19 251.6 mm to (245.0, 67.0), turned to -90 degrees
- moved J12 250.9 mm to (191.6, 45.1), turned to 83 degrees
- moved C25 248.7 mm to (248.6, 84.2), turned to 90 degrees
- moved D21 248.6 mm to (123.5, 131.8)
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Connections:
- C43 pad 2: Net-(C43-Pad2) -> Net-(U27-Pad2)
- H1 pad 1: (no net) -> GND
- H10 pad 1: (no net) -> GND
- H11 pad 1: (no net) -> GND
- H12 pad 1: (no net) -> GND
- H13 pad 1: (no net) -> GND
- H14 pad 1: (no net) -> GND
- H15 pad 1: (no net) -> GND
- H2 pad 1: (no net) -> GND
- H3 pad 1: (no net) -> GND
- H4 pad 1: (no net) -> GND
- H5 pad 1: (no net) -> GND
- H6 pad 1: (no net) -> GND
- H7 pad 1: (no net) -> GND
- H8 pad 1: (no net) -> GND
- H9 pad 1: (no net) -> GND
- J15 pad 6: Net-(C43-Pad2) -> Net-(U27-Pad2)
- U16 pad 6: /line_sensors/S2 -> GND
- U17 pad 2: /line_sensors/S3 -> /line_sensors/S2
- U18 pad 2: /line_sensors/S5 -> /line_sensors/S6
- U18 pad 6: GND -> /line_sensors/S8
- U19 pad 2: /line_sensors/S6 -> /line_sensors/S5
- U19 pad 6: /line_sensors/S7 -> /line_sensors/S3
- U20 pad 2: /line_sensors/S8 -> /line_sensors/S7
- U27 pad 2: Net-(C43-Pad1) -> Net-(U27-Pad2)
- U27 pad 3: Net-(C43-Pad2) -> Net-(C43-Pad1)
- U30 pad 2: Net-(C48-Pad1) -> Net-(C48-Pad2)
- U30 pad 3: Net-(C48-Pad2) -> Net-(C48-Pad1)
Routing:
- net GND: track 0.00 -> 1088.9 mm, vias 0 -> 60
- net +3V3: track 0.00 -> 72.3 mm
- net Net-(R73-Pad2): track 0.00 -> 52.6 mm
- net Net-(R72-Pad2): track 0.00 -> 52.0 mm
- net +VDC: track 0.00 -> 49.2 mm
- net /MODULE_SCL: track 0.00 -> 38.6 mm
- net /EXT4: track 0.00 -> 38.2 mm
- net /EXT2: track 0.00 -> 37.6 mm
- net /EXT6: track 0.00 -> 37.5 mm
- net /EXT10: track 0.00 -> 37.0 mm
- net /EXT8: track 0.00 -> 36.8 mm
- net /EXT0: track 0.00 -> 36.5 mm
- net /MODULE_SDA: track 0.00 -> 35.5 mm
- net /EXT5: track 0.00 -> 35.1 mm
- net /EXT3: track 0.00 -> 35.0 mm
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- added copper zone on F.Cu, net GND

Commit message: layout in progress
Parts:
- removed C31: 1u 50V, Capacitor_SMD:C_0603_1608Metric
- added J4: USB4085, GCT_USB4085:USB_C_Receptacle_GCT_USB4085, F.Cu at (165.5, 121.8)
- added Y1: 830056583, WE_830056583:830056583, F.Cu at (148.7, 68.7)
- added Y2: 830062558, WE_830062558:830062558, F.Cu at (155.4, 75.3)
- C4, D2, D3, Q4, Q7, R10, R12, R14, R16, R18, R27, R28, R29, R30, R31, R32, R33, R34, R35, R36, R37, R38, R39, R40, R41, R42, R43, R44, R45, R46, R47, R48, R49, R50, R51, R52, R53, R54, R55, R56, R6, R7, R9, U28, U29: moved to B.Cu
- R57, R58, R59, R63, R65, R70, R74, R75, R95: footprint Resistor_SMD:R_0805_2012Metric -> Resistor_SMD:R_0603_1608Metric_Pad0.98x0.95mm_HandSolder
- moved R92 289.2 mm to (247.6, 137.0), turned to -90 degrees
- moved R91 284.7 mm to (241.4, 134.1), turned to -90 degrees
- moved R87 282.7 mm to (249.8, 124.5), turned to 90 degrees
- moved R88 279.1 mm to (254.5, 120.8)
- moved R83 272.9 mm to (255.3, 107.5), turned to 90 degrees
- moved R84 270.6 mm to (259.2, 103.8)
- moved D23 267.5 mm to (223.5, 85.8), turned to 180 degrees
- moved R79 263.2 mm to (258.4, 92.6), turned to 90 degrees
- moved R80 262.0 mm to (262.6, 88.9)
- moved C34 261.4 mm to (227.0, 81.2), turned to 90 degrees
- moved U21 259.5 mm to (210.3, 87.6)
- moved L1 259.4 mm to (217.5, 85.6)
- moved R77 256.5 mm to (258.4, 82.6), turned to 90 degrees
- moved R78 255.8 mm to (262.6, 78.6)
- moved R105 255.6 mm to (224.9, 81.7), turned to 90 degrees
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Connections:
- SW3 pad 1: +3V0 -> +3V3
- SW4 pad 1: +3V0 -> +3V3
- U16 pad 7: /SENSOR_2 -> unconnected-(U16-Pad7)
- U17 pad 1: /SENSOR_3 -> /SENSOR_2
- U18 pad 1: /SENSOR_5 -> /SENSOR_6
- U18 pad 7: unconnected-(U18-Pad7) -> /SENSOR_8
- U19 pad 1: /SENSOR_6 -> /SENSOR_5
- U19 pad 7: /SENSOR_7 -> /SENSOR_3
- U20 pad 1: /SENSOR_8 -> /SENSOR_9
- U20 pad 2: /line_sensors/S7 -> /line_sensors/S9
- U20 pad 6: /line_sensors/S9 -> /line_sensors/S7
- U20 pad 7: /SENSOR_9 -> /SENSOR_7
Routing:
- net GND: track 1088.9 -> 2114.8 mm, vias 60 -> 91
- net +3V3: track 72.3 -> 757.7 mm, vias 0 -> 32
- net +VDC: track 49.2 -> 438.0 mm, vias 0 -> 14
- net /SENSOR_7: track 0.00 -> 208.9 mm, vias 0 -> 6
- net /SENSOR_9: track 0.00 -> 200.9 mm, vias 0 -> 6
- net /SENSOR_3: track 0.00 -> 178.1 mm, vias 0 -> 4
- net /SENSOR_5: track 0.00 -> 174.2 mm, vias 0 -> 4
- net /EXT5: track 35.1 -> 205.8 mm, vias 0 -> 4
- net Net-(R77-Pad1): track 0.00 -> 166.3 mm, vias 0 -> 11
- net /SENSOR_6: track 0.00 -> 160.5 mm, vias 0 -> 4
- net /SENSOR_8: track 0.00 -> 157.6 mm, vias 0 -> 6
- net /SENSOR_1: track 0.00 -> 155.8 mm, vias 0 -> 2
- net /SENSOR_2: track 0.00 -> 140.4 mm, vias 0 -> 2
- net /EXT2: track 37.6 -> 177.6 mm, vias 0 -> 4
- net /SENSOR_4: track 0.00 -> 139.1 mm, vias 0 -> 4
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
Commit message: routing done
Parts:
- added C31: 4.7u 10V, Capacitor_SMD:C_0805_2012Metric, F.Cu at (196.4, 52.6)
- added C64: 4.7u 10V, Capacitor_SMD:C_0805_2012Metric, F.Cu at (173.1, 47.7)
- added F4: 200mA SLOW, Fuse:Fuse_1206_3216Metric_Pad1.42x1.75mm_HandSolder, F.Cu at (159.9, 46.4)
- added F5: 200mA SLOW, Fuse:Fuse_1206_3216Metric_Pad1.42x1.75mm_HandSolder, F.Cu at (159.9, 48.8)
- C45, C46, C52, Q17, Q18, R109, R110, R111, R114, R115: moved to B.Cu
- moved J17 242.2 mm to (215.8, 109.4)
- moved J18 230.9 mm to (205.1, 103.7)
- moved C52 191.8 mm to (169.1, 126.8), turned to 180 degrees
- moved Q10 187.9 mm to (184.9, 93.7), turned to 180 degrees
- moved Q12 182.8 mm to (188.7, 82.0), turned to 180 degrees
- moved Q11 182.3 mm to (188.7, 85.5), turned to 180 degrees
- moved R60 173.7 mm to (188.8, 94.5), turned to 180 degrees
- moved R61 171.4 mm to (192.5, 86.3), turned to 180 degrees
- moved R62 169.1 mm to (192.6, 82.8), turned to 180 degrees
- moved C46 163.2 mm to (75.1, 93.7), turned to -90 degrees
- moved R57 158.9 mm to (188.8, 92.8), turned to 180 degrees
- moved R59 152.3 mm to (192.6, 81.2), turned to 180 degrees
- moved C45 150.7 mm to (75.5, 73.7), turned to 90 degrees
- moved R58 149.1 mm to (192.6, 84.7), turned to 180 degrees
- moved R8 148.8 mm to (137.9, 130.4), turned to 180 degrees
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Connections:
- J12 pad 1: +VDC -> Net-(J12-Pad1)
- J12 pad 2: +3V3 -> Net-(J12-Pad2)
- J13 pad 1: +VDC -> Net-(J12-Pad1)
- J13 pad 2: +3V3 -> Net-(J12-Pad2)
- J2 pad 1: +VDC -> Net-(J12-Pad1)
- J7 pad 10: /Peripherals/SD_DETECT -> /SD_DETECT
- R101 pad 2: /Peripherals/SD_DETECT -> /SD_DETECT
Routing:
- net GND: track 2114.8 -> 2671.2 mm, vias 91 -> 111
- net +3V3: track 757.7 -> 1301.6 mm, vias 32 -> 57
- net /UI/RED: track 110.7 -> 613.6 mm, vias 0 -> 11
- net /UI/GREEN: track 112.1 -> 613.4 mm, vias 2 -> 11
- net +VDC: track 438.0 -> 937.5 mm, vias 14 -> 30
- net /UI/BLUE: track 125.4 -> 624.0 mm, vias 2 -> 12
- net /PRH_SCL: track 0.00 -> 176.2 mm, vias 0 -> 13
- net /MODULE_SDA: track 125.2 -> 295.7 mm, vias 2 -> 4
- net /MODULE_SCL: track 129.8 -> 296.9 mm, vias 2 -> 5
- net /PRH_SDA: track 0.00 -> 165.2 mm, vias 0 -> 13
- net /SENSORS_ENABLE: track 2.28 -> 145.5 mm, vias 0 -> 8
- net /LED_DECOR_G: track 0.00 -> 136.6 mm, vias 0 -> 4
- net /SONAR_ENA: track 0.00 -> 132.3 mm, vias 0 -> 4
- net /MOTOR_L_PH: track 0.00 -> 123.6 mm, vias 0 -> 7
- net VBUS: track 48.1 -> 170.7 mm, vias 2 -> 5
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