File: BeamRider_MainBoard_v1.kicad_sch (KiCad schematic)
At the start: 24 parts, among them U1 RPR-220, U2 RPR-220, U3 RPR-220, U4 RPR-220, U5 RPR-220, U6 RPR-220, U7 RPR-220, U8 RPR-220, U9 RPR-220

Commit message: project structure
Parts:
- removed H1, H6: Caster_hole, MountingHole:MountingHole_2.2mm_M2_DIN965_Pad, symbol Mechanical:MountingHole
- removed H10, H4, H5, H9: Interface_hole, MountingHole:MountingHole_3.2mm_M3_DIN965_Pad, symbol Mechanical:MountingHole
- removed H11, H12, H13, H14, H15: Bumper_hole, MountingHole:MountingHole_3.2mm_M3_DIN965_Pad, symbol Mechanical:MountingHole
- removed H2, H3, H7, H8: Motor_hole, MountingHole:MountingHole_3.2mm_M3_DIN965_Pad, symbol Mechanical:MountingHole
- removed U1, U2, U3, U4, U5, U6, U7, U8, U9: RPR-220, RPR_220:RPR_220, symbol RPR_220:RPR-220
Other:
- added sheet Drive (drive.kicad_sch)
- added sheet External connectors (ext_conn.kicad_sch)
- added sheet MCU (MCU.kicad_sch)
- added sheet Peripherals (peripherals.kicad_sch)
- added sheet Power (power.kicad_sch)
- added sheet Structural (structural.kicad_sch)
- added sheet UI (UI.kicad_sch)
- added sheet line_sensors (line_sensors.kicad_sch)

Commit message: Schematic in progress
Other:
- sheet Drive ports: added BARREL_JACK_BUS, ENC_L_A, ENC_L_B, ENC_R_A, ENC_R_B, MOTOR_L_EN, MOTOR_L_PH, MOTOR_R_EN, MOTOR_R_PH; removed none
- sheet Power ports: added BARREL_JACK_BUS, USB_DM, USB_DP, USB_DP_PULL, VOLTAGE_MONITOR; removed none
- sheet UI ports: added BUTTON_1, BUTTON_2, DECORATIVE_BLUE, DECORATIVE_GREEN, DECORATIVE_RED, USER_BLUE, USER_GREEN, USER_RED; removed none
- sheet line_sensors ports: added SENSOR_1, SENSOR_2, SENSOR_3, SENSOR_4, SENSOR_5, SENSOR_6, SENSOR_7, SENSOR_8, SENSOR_9, SEN_EN; removed none

Commit message: schematic almost done
Parts:
- added R118, R119: 2k2 1%, Resistor_SMD:R_0603_1608Metric, symbol Device:R_Small
Connections:
- new net +3V3: R118.1, R119.1
- new net MODULE_SCL: R119.2
- new net MODULE_SDA: R118.2
Other:
- sheet External connectors ports: added EXT0, EXT1, EXT10, EXT11, EXT2, EXT3, EXT4, EXT5, EXT6, EXT7, EXT8, EXT9, EXT_SCL, EXT_SDA, MINI_A_0, MINI_A_1, MINI_A_2, MINI_A_3, MINI_A_4, MINI_A_SCL, MINI_A_SDA, MINI_B_0, MINI_B_1, MINI_B_2, MINI_B_3, MINI_B_4, MINI_B_SCL, MINI_B_SDA, PMOD_SCL, PMOD_SDA; removed none
- sheet MCU ports: added PA0, PA1, PA10, PA11, PA12, PA15, PA2, PA3, PA4, PA5, PA6, PA7, PA8, PA9, PB0, PB1, PB10, PB11, PB12, PB13, PB14, PB15, PB2, PB4, PB5, PB6, PB7, PB8, PB9, PC0, PC1, PC10, PC11, PC13, PC2, PC3, PC4, PC5, PC6, PC7, PC8, PC9, PD0, PD1, PD10, PD11, PD12, PD13, PD14, PD15, PD3, PD4, PD5, PD6, PD7, PD8, PD9, PE0, PE1, PE10, PE11, PE12, PE13, PE14, PE15, PE2, PE3, PE4, PE5, PE6, PE7, PE8, PE9; removed none
- sheet Peripherals ports: added ESP_CH_PD/EN, ESP_GPIO0, ESP_GPIO2, ESP_RST, ESP_RX, ESP_TX, INT_ACC, INT_MAG, PRH_SCL, PRH_SDA, SD_CLK, SD_CS, SD_DAT_IN, SD_DAT_OUT, SD_DETECT, SONAR_ECHO, SONAR_ENA, SONAR_TRIG; removed none
- sheet UI ports: added DEBUG_LED; removed none

Commit message: routing done
Changed lines of the file:
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@@
+    (stroke (width 0) (type default) (color 0 0 0 0))
+  )
+  (wire (pts (xy 227.33 156.21) (xy 234.95 156.21))
     (stroke (width 0) (type default) (color 0 0 0 0))
   )
@@
       (reference "#PWR020") (unit 1) (value "GND") (footprint "")
     )
-    (path "/4b8dabb8-2cfb-49bf-8c5b-3a99d0c3a8a8/771e6c9c-34a6-4359-8b37-b6a143b36f66"
-      (reference "#PWR021") (unit 1) (value "GND") (footprint "")
-    )
     (path "/4b8dabb8-2cfb-49bf-8c5b-3a99d0c3a8a8/6243bc15-ecc3-4552-a87e-1f8f92e261d8"
       (reference "#PWR022") (unit 1) (value "VBUS") (footprint "")
@@
       (reference "#PWR040") (unit 1) (value "GND") (footprint "")
     )
-    (path "/4b8dabb8-2cfb-49bf-8c5b-3a99d0c3a8a8/0652b275-e579-43ce-b0cc-0760aba2d8ad"
-      (reference "#PWR041") (unit 1) (value "+VDC") (footprint "")
-    )
     (path "/4b8dabb8-2cfb-49bf-8c5b-3a99d0c3a8a8/ec0a1da3-57d4-4e5f-bde5-dc7fd6a27852"
       (reference "#PWR042") (unit 1) (value "+VDC") (footprint "")
@@
       (reference "#PWR066") (unit 1) (value "GND") (footprint "")
     )
+    (path "/4ab7b350-0bbd-481f-bf8f-25946d061de1/c99efd65-35e7-4c4e-bf52-e1f49a4707ca"
+      (reference "#PWR067") (unit 1) (value "+3.3V") (footprint "")
+    )
+    (path "/4ab7b350-0bbd-481f-bf8f-25946d061de1/1a046fa3-62ff-4e33-b206-49e9db5880d5"
+      (reference "#PWR068") (unit 1) (value "GND") (footprint "")
+    )
     (path "/609946a4-476d-49df-a6f7-4168ea2d2a59/2920900a-ae53-4f88-8486-344de11b605a"
       (reference "#PWR069") (unit 1) (value "GND") (footprint "")
@@
       (reference "#PWR0139") (unit 1) (value "GND") (footprint "")
     )
+    (path "/4ab7b350-0bbd-481f-bf8f-25946d061de1/082d9f80-3872-434f-b251-a15648bc3117"
+      (reference "#PWR0140") (unit 1) (value "+VDC") (footprint "")
+    )
     (path "/4b62ad27-c3c4-44dc-845c-a46dc33e6d80/c54d0d97-d449-4a89-acc7-cdbfeb24699f"
       (reference "#PWR0141") (unit 1) (value "GND") (footprint "")
@@
       (reference "#PWR0217") (unit 1) (value "GND") (footprint "")
     )
-    (path "/4ab7b350-0bbd-481f-bf8f-25946d061de1/3ded34e9-0846-4f4a-9d71-ae8dd56e3520"
-      (reference "#PWR0218") (unit 1) (value "+VDC") (footprint "")
-    )
-    (path "/4ab7b350-0bbd-481f-bf8f-25946d061de1/a4f675ed-aff1-4040-bb98-6cffdfd0eca9"
-      (reference "#PWR0219") (unit 1) (value "+3.3V") (footprint "")
+    (path "/4ab7b350-0bbd-481f-bf8f-25946d061de1/ac13453f-ee4f-4765-9ed7-3b065fa4354f"
+      (reference "#PWR0218") (unit 1) (value "GND") (footprint "")
     )
     (path "/4ab7b350-0bbd-481f-bf8f-25946d061de1/e8ec1a98-fdb7-4d51-b575-e99eb88849fc"
       (reference "#PWR0220") (unit 1) (value "GND") (footprint "")
     )
-    (path "/4ab7b350-0bbd-481f-bf8f-25946d061de1/19f4091c-4abf-41a2-9300-92aef45221c4"
-      (reference "#PWR0221") (unit 1) (value "+VDC") (footprint "")
-    )
-    (path "/4ab7b350-0bbd-481f-bf8f-25946d061de1/9f1990d4-63b0-4a98-acbf-5feae449dfbf"
-      (reference "#PWR0222") (unit 1) (value "+3.3V") (footprint "")
-    )
     (path "/4ab7b350-0bbd-481f-bf8f-25946d061de1/ad8017be-2057-4cb4-911f-1951039232b5"
       (reference "#PWR0223") (unit 1) (value "+3.3V") (footprint "")
@@
       (reference "#PWR0242") (unit 1) (value "+3.3V") (footprint "")
     )
+    (path "/4ab7b350-0bbd-481f-bf8f-25946d061de1/68486ee7-787f-44d0-9354-6c16e63b3fd7"
+      (reference "#PWR?") (unit 1) (value "GND") (footprint "")
+    )
     (path "/4b8dabb8-2cfb-49bf-8c5b-3a99d0c3a8a8/546d9f29-0814-4854-a572-2f8c235571d4"
       (reference "BT1") (unit 1) (value "LiION_18650") (footprint "Battery:BatteryHolder_Keystone_1042_1x18650")
@@
       (reference "C30") (unit 1) (value "100n 50V") (footprint "Capacitor_SMD:C_0603_1608Metric")
     )
+    (path "/4ab7b350-0bbd-481f-bf8f-25946d061de1/91cb798b-6a7b-497d-91cc-fd211d0ee226"
+      (reference "C31") (unit 1) (value "4.7u 10V") (footprint "Capacitor_SMD:C_0805_2012Metric")
+    )
     (path "/4b62ad27-c3c4-44dc-845c-a46dc33e6d80/fef1cf92-1476-4e8b-8e4e-7e0f49784480"
       (reference "C32") (unit 1) (value "10u 25V") (footprint "Capacitor_SMD:C_0805_2012Metric")
@@
       (reference "C63") (unit 1) (value "1u 10V") (footprint "Capacitor_SMD:C_0603_1608Metric_Pad1.08x0.95mm_HandSolder")
     )
+    (path "/4ab7b350-0bbd-481f-bf8f-25946d061de1/7db8f754-6da0-4fc1-b407-da303efe430d"
+      (reference "C64") (unit 1) (value "4.7u 10V") (footprint "Capacitor_SMD:C_0805_2012Metric")
+    )
     (path "/609946a4-476d-49df-a6f7-4168ea2d2a59/3408444a-2f91-4f6a-b27d-7fd42fbe6a0f"
       (reference "D1") (unit 1) (value "RGB_LED") (footprint "LED_SMD:LED_RGB_Wuerth-PLCC4_3.2x2.8mm_150141M173100")
@@
       (reference "F3") (unit 1) (value "5A SLOW") (footprint "Fuse:Fuse_1206_3216Metric_Pad1.42x1.75mm_HandSolder")
     )
+    (path "/4ab7b350-0bbd-481f-bf8f-25946d061de1/8df3e3e5-0fec-4928-ac40-de2f72499c38"
+      (reference "F4") (unit 1) (value "200mA SLOW") (footprint "Fuse:Fuse_1206_3216Metric_Pad1.42x1.75mm_HandSolder")
+    )
+    (path "/4ab7b350-0bbd-481f-bf8f-25946d061de1/8e41b0a5-b1a1-4478-975d-b9a691530b53"
+      (reference "F5") (unit 1) (value "200mA SLOW") (footprint "Fuse:Fuse_1206_3216Metric_Pad1.42x1.75mm_HandSolder")
+    )
     (path "/75dee642-618b-4ed2-b6e1-8db2e50d8e51/fb011f35-788d-4eac-9fff-bca57cbea1fa"
       (reference "H1") (unit 1) (value "Caster_hole") (footprint "MountingHole:MountingHole_2.2mm_M2_DIN965_Pad")
@@
       (reference "J1") (unit 1) (value "Barrel_Jack") (footprint "Connector_BarrelJack:BarrelJack_GCT_DCJ200-10-A_Horizontal")
     )
-    (path "/4b8dabb8-2cfb-49bf-8c5b-3a99d0c3a8a8/729dbb87-c21a-4cf6-9ff8-46ee599719bd"
+    (path "/4ab7b350-0bbd-481f-bf8f-25946d061de1/bf0b47a2-7ac7-4cbd-9fe8-471bba234e8d"
       (reference "J2") (unit 1) (value "POWER_OUT") (footprint "TerminalBlock:TerminalBlock_bornier-2_P5.08mm")
     )
