File: BeamRider_MainBoard_v1.kicad_sch (KiCad schematic)
At the start: 2 parts

Commit message: schematics update
Other:
- company: (none) -> Wrocław University of Science and Technology
- title: (none) -> Top-level signal interconnect
Changed lines of the file:
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@@
 (kicad_sch (version 20211123) (generator eeschema)
   (paper "A4")
+  (title_block
+    (title "Top-level signal interconnect")
+    (date "2023-04-04")
+    (rev "1")
+    (company "Wrocław University of Science and Technology")
+    (comment 1 "Opensource educational robotic platform")
+    (comment 2 "Author: Jakub Mnich (jakub.mnich@pwr.edu.pl)")
+  )
   (wire (pts (xy 46.99 43.18) (xy 49.53 43.18))
     (stroke (width 0) (type default) (color 0 0 0 0))
