File: MCU.kicad_sch (KiCad schematic)
At the start: 1 part

Commit message: components selection
Parts:
- added C1: 100n 50V, Capacitor_SMD:C_0603_1608Metric_Pad1.08x0.95mm_HandSolder, symbol Device:C_Small
- added SW1: RST, Button_Switch_THT:SW_PUSH_6mm_H5mm, symbol Switch:SW_Push
Connections:
- new net GND: C1.2, SW1.2
- new net NRST: C1.1, SW1.1
Changed lines of the file:
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@@
 (kicad_sch (version 20211123) (generator eeschema)
   (paper "A4")
+  (junction (at 207.01 66.04) (diameter 0) (color 0 0 0 0)
+  )
+  (wire (pts (xy 207.01 72.39) (xy 207.01 73.66))
+    (stroke (width 0) (type default) (color 0 0 0 0))
+  )
+  (wire (pts (xy 207.01 66.04) (xy 207.01 67.31))
+    (stroke (width 0) (type default) (color 0 0 0 0))
+  )
+  (wire (pts (xy 220.98 66.04) (xy 222.25 66.04))
+    (stroke (width 0) (type default) (color 0 0 0 0))
+  )
+  (wire (pts (xy 222.25 66.04) (xy 222.25 73.66))
+    (stroke (width 0) (type default) (color 0 0 0 0))
+  )
+  (wire (pts (xy 207.01 66.04) (xy 210.82 66.04))
+    (stroke (width 0) (type default) (color 0 0 0 0))
+  )
+  (wire (pts (xy 201.93 66.04) (xy 207.01 66.04))
+    (stroke (width 0) (type default) (color 0 0 0 0))
+  )
+  (label "NRST" (at 201.93 66.04 0)
+    (effects (font (size 1.27 1.27)) (justify left bottom))
+  )
+  (symbol (lib_id "Switch:SW_Push") (at 215.9 66.04 0) (unit 1)
+    (in_bom yes) (on_board yes)
+    (property "Reference" "SW1" (id 0) (at 215.9 60.96 0))
+    (property "Value" "RST" (id 1) (at 213.36 63.5 0))
+    (property "Footprint" "Button_Switch_THT:SW_PUSH_6mm_H5mm" (id 2) (at 215.9 60.96 0)
+      (effects (font (size 1.27 1.27)) hide)
+    )
+    (property "Datasheet" "~" (id 3) (at 215.9 60.96 0)
+      (effects (font (size 1.27 1.27)) hide)
+    )
+    (pin "1")
+    (pin "2")
+  )
+  (symbol (lib_id "power:GND") (at 222.25 73.66 0) (unit 1)
+    (in_bom yes) (on_board yes)
+    (property "Reference" "#PWR02" (id 0) (at 222.25 80.01 0)
+      (effects (font (size 1.27 1.27)) hide)
+    )
+    (property "Value" "GND" (id 1) (at 222.25 77.47 0))
+    (property "Footprint" "" (id 2) (at 222.25 73.66 0)
+      (effects (font (size 1.27 1.27)) hide)
+    )
+    (property "Datasheet" "" (id 3) (at 222.25 73.66 0)
+      (effects (font (size 1.27 1.27)) hide)
+    )
+    (pin "1")
+  )
+  (symbol (lib_id "power:GND") (at 207.01 73.66 0) (unit 1)
+    (in_bom yes) (on_board yes)
+    (property "Reference" "#PWR01" (id 0) (at 207.01 80.01 0)
+      (effects (font (size 1.27 1.27)) hide)
+    )
+    (property "Value" "GND" (id 1) (at 207.01 77.47 0))
+    (property "Footprint" "" (id 2) (at 207.01 73.66 0)
+      (effects (font (size 1.27 1.27)) hide)
+    )
+    (property "Datasheet" "" (id 3) (at 207.01 73.66 0)
+      (effects (font (size 1.27 1.27)) hide)
+    )
+    (pin "1")
+  )
   (symbol (lib_id "MCU_ST_STM32F4:STM32F407VETx") (at 99.06 107.95 0) (unit 1)
     (in_bom yes) (on_board yes) (fields_autoplaced)
@@
     (pin "99")
   )
+  (symbol (lib_id "Device:C_Small") (at 207.01 69.85 0) (mirror y) (unit 1)
+    (in_bom yes) (on_board yes)
+    (property "Reference" "C1" (id 0) (at 213.36 68.58 0)
+      (effects (font (size 1.27 1.27)) (justify left))
+    )
+    (property "Value" "100n 50V" (id 1) (at 218.44 71.12 0)
+      (effects (font (size 1.27 1.27)) (justify left))
+    )
+    (property "Footprint" "Capacitor_SMD:C_0603_1608Metric_Pad1.08x0.95mm_HandSolder" (id 2) (at 207.01 69.85 0)
+      (effects (font (size 1.27 1.27)) hide)
+    )
+    (property "Datasheet" "~" (id 3) (at 207.01 69.85 0)
+      (effects (font (size 1.27 1.27)) hide)
+    )
+    (pin "1")
+    (pin "2")
+  )
 )

Commit message: Schematic in progress
Parts:
- MCU1: value STM32F407VETx -> STM32F407VGT6; M (none) -> ST; MPN (none) -> STM32F407VGT6
Changed lines of the file:
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@@
       (effects (font (size 1.27 1.27)) (justify left))
     )
-    (property "Value" "STM32F407VETx" (id 1) (at 106.1594 179.07 0)
+    (property "Value" "STM32F407VGT6" (id 1) (at 106.1594 179.07 0)
       (effects (font (size 1.27 1.27)) (justify left))
     )
@@
       (effects (font (size 1.27 1.27)) hide)
     )
+    (property "M" "ST" (id 4) (at 99.06 107.95 0)
+      (effects (font (size 1.27 1.27)) hide)
+    )
+    (property "MPN" "STM32F407VGT6" (id 5) (at 99.06 107.95 0)
+      (effects (font (size 1.27 1.27)) hide)
+    )

Commit message: schematic almost done
Parts:
- added C16, C17: 20p 10V, Capacitor_SMD:C_0603_1608Metric_Pad1.08x0.95mm_HandSolder, symbol Device:C_Small
- added C18, C19: 2u2 6.3V, Capacitor_SMD:C_0603_1608Metric_Pad1.08x0.95mm_HandSolder, symbol Device:C_Small
- added C20, C21, C53, C54, C55, C56, C57, C58, C59: 100n 50V, Capacitor_SMD:C_0603_1608Metric, symbol Device:C_Small
- added C22, C23: 16p 10V, Capacitor_SMD:C_0603_1608Metric_Pad1.08x0.95mm_HandSolder, symbol Device:C_Small
- added C60, C61, C62: 4.7u 10V, Capacitor_SMD:C_0805_2012Metric, symbol Device:C_Small
- added C63: 1u 10V, Capacitor_SMD:C_0603_1608Metric_Pad1.08x0.95mm_HandSolder, symbol Device:C_Small
- added J14: AUX_PROG, Connector_PinHeader_2.54mm:PinHeader_1x06_P2.54mm_Vertical, symbol Connector_Generic:Conn_01x06
- added J17: UART_Bridge, Connector_PinHeader_2.54mm:PinHeader_1x03_P2.54mm_Vertical, symbol Connector_Generic:Conn_01x03
- added J18: I2C_Bridge, Connector_PinHeader_2.54mm:PinHeader_1x03_P2.54mm_Vertical, symbol Connector_Generic:Conn_01x03
- added J5: BOOT_SEL, Connector_PinHeader_2.54mm:PinHeader_1x03_P2.54mm_Vertical, symbol Connector_Generic:Conn_01x03
- added TP2: TestPoint, TestPoint:TestPoint_THTPad_D2.5mm_Drill1.2mm, symbol Connector:TestPoint
- added U31: STLINK_V3MODS, STLINK_V3MODS:STLINK-V3MODS, symbol STLINK_V3MODS:STLINK_V3MODS
- added Y1: 830056583, WE_830056583:830056583, symbol Device:Crystal_GND24
- added Y2: 830062558, WE_830062558:830062558, symbol Device:Crystal_Small
Connections:
- net GND: now also MCU1.10 (VSS), MCU1.20 (VSSA), MCU1.27 (VSS), MCU1.74 (VSS), MCU1.99 (VSS), C16.1, C17.1, C18.1, C19.1, C20.2, C21.2, C22.2, C23.2, C53.2, C54.2, C55.2, C56.2, C57.2, C58.2, C59.2, C60.2, C61.2, C62.2, C63.2, J14.3 (Pin_3), J17.1 (Pin_1), J18.1 (Pin_1), J5.3 (Pin_3), U31.24 (GND), U31.26 (GND), U31.27 (GND), U31.29 (GND), U31.5 (GNDDetect), U31.8 (GND), Y1.2, Y1.4
- net NRST: now also MCU1.14 (NRST), J14.5 (Pin_5), U31.31 (T_NRST)
- net PE2: now reaches MCU1.1 (PE2)
- net +3V3: now reaches MCU1.100 (VDD)
- net +3V3: now also MCU1.11 (VDD), MCU1.19 (VDD), MCU1.21 (VREF+), MCU1.22 (VDDA), MCU1.28 (VDD), MCU1.50 (VDD), MCU1.6 (VBAT), MCU1.75 (VDD), C20.1, C21.1, C53.1, C54.1, C55.1, C56.1, C57.1, C58.1, C59.1, C60.1, C61.1, C62.1, C63.1, J14.1 (Pin_1), J5.1 (Pin_1), U31.30 (T_VCC)
- net at MCU1.12 (PH0): now also C16.2, Y1.3
- net at MCU1.13 (PH1): now also C17.2, Y1.1
- net PC0: now reaches MCU1.15 (PC0)
- net PC1: now reaches MCU1.16 (PC1)
- net PC2: now reaches MCU1.17 (PC2)
- net PC3: now reaches MCU1.18 (PC3)
- net PE3: now reaches MCU1.2 (PE3)
- net PA0: now reaches MCU1.23 (PA0)
- net PA1: now reaches MCU1.24 (PA1)
- net PA2: now reaches MCU1.25 (PA2)
- net PA3: now reaches MCU1.26 (PA3)
- net PA4: now reaches MCU1.29 (PA4)
- net PE4: now reaches MCU1.3 (PE4)
- net PA5: now reaches MCU1.30 (PA5)
- net PA6: now reaches MCU1.31 (PA6)
- net PA7: now reaches MCU1.32 (PA7)
- net PC4: now reaches MCU1.33 (PC4)
- net PC5: now reaches MCU1.34 (PC5)
- net PB0: now reaches MCU1.35 (PB0)
- net PB1: now reaches MCU1.36 (PB1)
- net PB2: now reaches MCU1.37 (PB2)
- net PE7: now reaches MCU1.38 (PE7)
- net PE8: now reaches MCU1.39 (PE8)
- net PE5: now reaches MCU1.4 (PE5)
- net PE9: now reaches MCU1.40 (PE9)
- net PE10: now reaches MCU1.41 (PE10)
- net PE11: now reaches MCU1.42 (PE11)
- net PE12: now reaches MCU1.43 (PE12)
- net PE13: now reaches MCU1.44 (PE13)
- net PE14: now reaches MCU1.45 (PE14)
- net PE15: now reaches MCU1.46 (PE15)
- net PB10: now reaches MCU1.47 (PB10)
- net PB11: now reaches MCU1.48 (PB11)
- net at MCU1.49 (VCAP_1): now also C18.2
- net PE6: now reaches MCU1.5 (PE6)
- net PB12: now reaches MCU1.51 (PB12)
- net PB13: now reaches MCU1.52 (PB13)
- net PB14: now reaches MCU1.53 (PB14)
- net PB15: now reaches MCU1.54 (PB15)
- net PD8: now reaches MCU1.55 (PD8)
- net PD9: now reaches MCU1.56 (PD9)
- net PD10: now reaches MCU1.57 (PD10)
- net PD11: now reaches MCU1.58 (PD11)
- net PD12: now reaches MCU1.59 (PD12)
- net PD13: now reaches MCU1.60 (PD13)
- net PD14: now reaches MCU1.61 (PD14)
- net PD15: now reaches MCU1.62 (PD15)
- net PC6: now reaches MCU1.63 (PC6)
- net PC7: now reaches MCU1.64 (PC7)
- net PC8: now reaches MCU1.65 (PC8)
- net PC9: now reaches MCU1.66 (PC9)
- net PA8: now reaches MCU1.67 (PA8)
- net PA9: now reaches MCU1.68 (PA9)
- net PA10: now reaches MCU1.69 (PA10)
- net PC13: now reaches MCU1.7 (PC13)
- net PA11: now reaches MCU1.70 (PA11)
- net PA12: now reaches MCU1.71 (PA12)
- net STLINK_SWDIO: now reaches MCU1.72 (PA13)
- net STLINK_SWDIO: now also J14.4 (Pin_4), U31.4 (T_JTMS/T_SWDIO)
- net at MCU1.73 (VCAP_2): now also C19.2
- net STLINK_SWCLK: now reaches MCU1.76 (PA14)
- net STLINK_SWCLK: now also J14.2 (Pin_2), U31.13 (T_JCLK/T_SWCLK)
- net PA15: now reaches MCU1.77 (PA15)
- net PC10: now reaches MCU1.78 (PC10)
- net PC11: now reaches MCU1.79 (PC11)
- net at MCU1.8 (PC14): now also C22.1, Y2.1
- net STLINK_VCP_RX: now reaches MCU1.80 (PC12)
- net STLINK_VCP_RX: now also U31.15 (T_VCP_RX)
- net PD0: now reaches MCU1.81 (PD0)
- net PD1: now reaches MCU1.82 (PD1)
- net STLINK_VCP_TX: now reaches MCU1.83 (PD2)
- net STLINK_VCP_TX: now also U31.12 (T_VCP_TX)
- net PD3: now reaches MCU1.84 (PD3)
- net PD4: now reaches MCU1.85 (PD4)
- net PD5: now reaches MCU1.86 (PD5)
- net PD6: now reaches MCU1.87 (PD6)
- net PD7: now reaches MCU1.88 (PD7)
- net STLINK_SWO: now reaches MCU1.89 (PB3)
- net STLINK_SWO: now also J14.6 (Pin_6), U31.6 (T_JTDO/T_SWO)
- net at MCU1.9 (PC15): now also C23.1, Y2.2
- net PB4: now reaches MCU1.90 (PB4)
- net PB5: now reaches MCU1.91 (PB5)
- net PB6: now reaches MCU1.92 (PB6)
- net PB7: now reaches MCU1.93 (PB7)
- net at MCU1.94 (BOOT0): now also J5.2 (Pin_2)
- net PB8: now reaches MCU1.95 (PB8)
- net PB9: now reaches MCU1.96 (PB9)
- net PE0: now reaches MCU1.97 (PE0)
- net PE1: now reaches MCU1.98 (PE1)
- new net: J17.2 (Pin_2), U31.11 (Bridge_UART_TX)
- new net: J17.3 (Pin_3), U31.1 (Bridge_UART_RX)
- new net: TP2.1, U31.32 (T_SW_DIR)
- new net: J18.2 (Pin_2), U31.17 (Bridge_I2C_SDA)
- new net: J18.3 (Pin_3), U31.16 (Bridge_I2C_SCL)
- no-connect marks 0 -> 14
Other:
- note added: "10MHz"
- note added: "Backup interface"
- note added: "MCU"
- note added: "STLink"
- moved on the sheet: C1, MCU1, SW1

Commit message: Layout in progress
Parts:
- SW1: footprint Button_Switch_THT:SW_PUSH_6mm_H5mm -> Button_Switch_SMD:SW_Push_1P1T_NO_6x6mm_H9.5mm
Changed lines of the file:
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@@
     (property "Reference" "SW1" (id 0) (at 54.61 25.4 0))
     (property "Value" "RST" (id 1) (at 52.07 27.94 0))
-    (property "Footprint" "Button_Switch_THT:SW_PUSH_6mm_H5mm" (id 2) (at 54.61 25.4 0)
+    (property "Footprint" "Button_Switch_SMD:SW_Push_1P1T_NO_6x6mm_H9.5mm" (id 2) (at 54.61 25.4 0)
       (effects (font (size 1.27 1.27)) hide)
     )

Commit message: layout in progress
Changed lines of the file:
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@@
   (symbol (lib_id "Device:C_Small") (at 27.94 85.09 90) (unit 1)
     (in_bom yes) (on_board yes)
-    (property "Reference" "C16" (id 0) (at 31.75 83.82 90)
+    (property "Reference" "C16" (id 0) (at 33.02 83.82 90)
       (effects (font (size 1.27 1.27)) (justify left))
     )
@@
   (symbol (lib_id "Device:C_Small") (at 27.94 95.25 90) (unit 1)
     (in_bom yes) (on_board yes)
-    (property "Reference" "C17" (id 0) (at 31.75 93.98 90)
+    (property "Reference" "C17" (id 0) (at 33.02 93.98 90)
       (effects (font (size 1.27 1.27)) (justify left))
     )
@@
   (symbol (lib_id "Device:C_Small") (at 58.42 62.23 90) (mirror x) (unit 1)
     (in_bom yes) (on_board yes)
-    (property "Reference" "C18" (id 0) (at 62.23 60.96 90)
+    (property "Reference" "C18" (id 0) (at 63.5 60.96 90)
       (effects (font (size 1.27 1.27)) (justify left))
     )
@@
   (symbol (lib_id "Device:C_Small") (at 58.42 67.31 90) (mirror x) (unit 1)
     (in_bom yes) (on_board yes)
-    (property "Reference" "C19" (id 0) (at 62.23 66.04 90)
-      (effects (font (size 1.27 1.27)) (justify left))
-    )
+    (property "Reference" "C19" (id 0) (at 63.5 66.04 90)
+      (effects (font (size 1.27 1.27)) (justify left))
+    )

Commit message: schematics update
Other:
- company: (none) -> Wrocław University of Science and Technology
- title: (none) -> Microcontroller
Changed lines of the file:
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@@
 (kicad_sch (version 20211123) (generator eeschema)
   (paper "A4")
+  (title_block
+    (title "Microcontroller")
+    (date "2023-04-04")
+    (rev "1")
+    (company "Wrocław University of Science and Technology")
+    (comment 1 "Opensource educational robotic platform")
+    (comment 2 "Author: Jakub Mnich (jakub.mnich@pwr.edu.pl)")
+  )
   (junction (at 72.39 72.39) (diameter 0) (color 0 0 0 0)
   )
