File: drive.kicad_sch (KiCad schematic)
At the start: 0 parts

Commit message: Schematic in progress
Parts:
- added C? (x2): 1u 50V, Capacitor_SMD:C_0603_1608Metric, symbol Device:C_Small
- added C? (x6): 100n 50V, Capacitor_SMD:C_0603_1608Metric, symbol Device:C_Small
- added C? (x2): 22u 16V, Capacitor_SMD:C_1206_3216Metric, symbol Device:C_Small
- added C? (x2): 220p 50V, Capacitor_SMD:C_0603_1608Metric, symbol Device:C_Small
- added J?: Motor_R, Connector_PinHeader_2.54mm:PinHeader_1x06_P2.54mm_Vertical, symbol Connector_Generic:Conn_01x06
- added J?: Motor_L, Connector_PinHeader_2.54mm:PinHeader_1x06_P2.54mm_Vertical, symbol Connector_Generic:Conn_01x06
- added Q? (x2): 2N7002NXAK, Package_TO_SOT_SMD:SOT-23, symbol Transistor_FET:2N7002
- added R? (x3): 10k 1%, Resistor_SMD:R_0603_1608Metric_Pad0.98x0.95mm_HandSolder, symbol Device:R_Small
- added R? (x2): 0R 5% (DNP), Resistor_SMD:R_0603_1608Metric_Pad0.98x0.95mm_HandSolder, symbol Device:R_Small
- added R? (x2): 100R 1%, Resistor_SMD:R_0603_1608Metric_Pad0.98x0.95mm_HandSolder, symbol Device:R_Small
- added R? (x2): 0R 5%, Resistor_SMD:R_0603_1608Metric_Pad0.98x0.95mm_HandSolder, symbol Device:R_Small
- added U? (x6): 74HC2G08DP,125, Package_SO:TSSOP-8_3x3mm_P0.65mm, symbol 74HC2G08DP:74HC2G08DP,125
- added U? (x2): DRV8212DSG, Package_SON:WSON-8-1EP_2x2mm_P0.5mm_EP0.9x1.6mm_ThermalVias, symbol DRV8212:DRV8212DSG
Connections:
- new net: Q?.1 (G), R?.1, R?.1 (x2)
- new net: R?.1, R?.2, U?.7 (MODE) (x2)
- new net: C?.1, J?.1 (Pin_1), U?.2 (OUT1) (x2)
- new net: C?.2, J?.6 (Pin_6), U?.3 (OUT2) (x2)
- new net +3V3: C?.1, C?.1, C?.1, C?.1, C?.2, C?.2, J?.5 (Pin_5), J?.5 (Pin_5), R?.1, R?.1, R?.1, U?.8 (VCC), U?.8 (VCC), U?.8 (VCC), U?.8 (VCC)
- new net +VDC: C?.1, C?.1, C?.1, C?.1, U?.1 (VM), U?.1 (VM)
- new net BARREL_JACK_BUS: R?.2
- new net CUTOFF: Q?.3 (D), Q?.3 (D), R?.2, U?.2 (1B), U?.2 (1B), U?.6 (2B), U?.6 (2B)
- new net ENC_L_A: J?.3 (Pin_3)
- new net ENC_L_B: J?.4 (Pin_4)
- new net ENC_R_A: J?.3 (Pin_3)
- new net ENC_R_B: J?.4 (Pin_4)
- new net GND: C?.1, C?.1, C?.2, C?.2, C?.2, C?.2, C?.2, C?.2, C?.2, C?.2, J?.2 (Pin_2), J?.2 (Pin_2), Q?.2 (S), Q?.2 (S), R?.2, R?.2, R?.2, R?.2, U?.4 (GND), U?.4 (GND), U?.4 (GND), U?.4 (GND), U?.9 (TH_GND), U?.9 (TH_GND)
- new net L_EN: U?.3 (2Y), U?.5 (IN2/EN)
- new net L_PH: U?.6 (IN1/PH), U?.7 (1Y)
- new net MOTOR_L_EN: U?.5 (2A)
- new net MOTOR_L_PH: U?.1 (1A)
- new net MOTOR_R_EN: U?.5 (2A)
- new net MOTOR_R_PH: U?.1 (1A)
- new net R_EN: U?.3 (2Y), U?.5 (IN2/EN)
- new net R_PH: U?.6 (IN1/PH), U?.7 (1Y)
- new net VBUS: R?.2
Other:
- note added: "H-Bridges and motor connections"
- note added: "Safety cutoff for H-bridges"
- note added: "Used for disabling motors when external charger is connected."

Commit message: schematic almost done
Parts:
- gave numbers to parts that had none: 29

Commit message: Layout in progress
Connections:
- net at C48.1, J16.1 (Pin_1): now also U30.3 (OUT2); no longer U30.2 (OUT1)
- net at C48.2, J16.6 (Pin_6): now also U30.2 (OUT1); no longer U30.3 (OUT2)
- net at C43.1, J15.1 (Pin_1): now also U27.3 (OUT2); no longer U27.2 (OUT1)
- net at C43.2, J15.6 (Pin_6): now also U27.2 (OUT1); no longer U27.3 (OUT2)

Commit message: schematics update
Other:
- company: (none) -> Wrocław University of Science and Technology
- title: (none) -> Motors' control
Changed lines of the file:
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@@
 (kicad_sch (version 20211123) (generator eeschema)
   (paper "A4")
+  (title_block
+    (title "Motors' control")
+    (date "2023-04-04")
+    (rev "1")
+    (company "Wrocław University of Science and Technology")
+    (comment 1 "Opensource educational robotic platform")
+    (comment 2 "Author: Jakub Mnich (jakub.mnich@pwr.edu.pl)")
+  )
   (junction (at 214.63 80.01) (diameter 0) (color 0 0 0 0)
   )
