File: ext_conn.kicad_sch (KiCad schematic)
At the start: 0 parts

Commit message: Schematic in progress
Parts:
- added J?: PMOD, Connector_PinSocket_2.54mm:PinSocket_2x06_P2.54mm_Vertical, symbol Connector_Generic:Conn_02x06_Odd_Even
- added J? (x2): IDC_2x5, Connector_IDC:IDC-Header_2x05_P2.54mm_Vertical, symbol Connector_Generic:Conn_02x05_Odd_Even
- added J?: IDC_2x10, Connector_IDC:IDC-Header_2x10_P2.54mm_Vertical, symbol Connector_Generic:Conn_02x10_Odd_Even
Changed lines of the file:
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@@
 (kicad_sch (version 20211123) (generator eeschema)
   (paper "A4")
+  (symbol (lib_id "Connector_Generic:Conn_02x06_Odd_Even") (at 203.2 62.23 0) (unit 1)
+    (in_bom yes) (on_board yes) (fields_autoplaced)
+    (property "Reference" "J?" (id 0) (at 204.47 50.8 0))
+    (property "Value" "PMOD" (id 1) (at 204.47 53.34 0))
+    (property "Footprint" "Connector_PinSocket_2.54mm:PinSocket_2x06_P2.54mm_Vertical" (id 2) (at 203.2 62.23 0)
+      (effects (font (size 1.27 1.27)) hide)
+    )
+    (property "Datasheet" "~" (id 3) (at 203.2 62.23 0)
+      (effects (font (size 1.27 1.27)) hide)
+    )
+    (pin "1")
+    (pin "10")
+    (pin "11")
+    (pin "12")
+    (pin "2")
+    (pin "3")
+    (pin "4")
+    (pin "5")
+    (pin "6")
+    (pin "7")
+    (pin "8")
+    (pin "9")
+  )
+  (symbol (lib_id "Connector_Generic:Conn_02x05_Odd_Even") (at 167.64 66.04 0) (unit 1)
+    (in_bom yes) (on_board yes) (fields_autoplaced)
+    (property "Reference" "J?" (id 0) (at 168.91 54.61 0))
+    (property "Value" "IDC_2x5" (id 1) (at 168.91 57.15 0))
+    (property "Footprint" "Connector_IDC:IDC-Header_2x05_P2.54mm_Vertical" (id 2) (at 167.64 66.04 0)
+      (effects (font (size 1.27 1.27)) hide)
+    )
+    (property "Datasheet" "~" (id 3) (at 167.64 66.04 0)
+      (effects (font (size 1.27 1.27)) hide)
+    )
+    (pin "1")
+    (pin "10")
+    (pin "2")
+    (pin "3")
+    (pin "4")
+    (pin "5")
+    (pin "6")
+    (pin "7")
+    (pin "8")
+    (pin "9")
+  )
+  (symbol (lib_id "Connector_Generic:Conn_02x10_Odd_Even") (at 87.63 71.12 0) (unit 1)
+    (in_bom yes) (on_board yes) (fields_autoplaced)
+    (property "Reference" "J?" (id 0) (at 88.9 54.61 0))
+    (property "Value" "IDC_2x10" (id 1) (at 88.9 57.15 0))
+    (property "Footprint" "Connector_IDC:IDC-Header_2x10_P2.54mm_Vertical" (id 2) (at 87.63 71.12 0)
+      (effects (font (size 1.27 1.27)) hide)
+    )
+    (property "Datasheet" "~" (id 3) (at 87.63 71.12 0)
+      (effects (font (size 1.27 1.27)) hide)
+    )
+    (pin "1")
+    (pin "10")
+    (pin "11")
+    (pin "12")
+    (pin "13")
+    (pin "14")
+    (pin "15")
+    (pin "16")
+    (pin "17")
+    (pin "18")
+    (pin "19")
+    (pin "2")
+    (pin "20")
+    (pin "3")
+    (pin "4")
+    (pin "5")
+    (pin "6")
+    (pin "7")
+    (pin "8")
+    (pin "9")
+  )
+  (symbol (lib_id "Connector_Generic:Conn_02x05_Odd_Even") (at 148.59 66.04 0) (unit 1)
+    (in_bom yes) (on_board yes) (fields_autoplaced)
+    (property "Reference" "J?" (id 0) (at 149.86 54.61 0))
+    (property "Value" "IDC_2x5" (id 1) (at 149.86 57.15 0))
+    (property "Footprint" "Connector_IDC:IDC-Header_2x05_P2.54mm_Vertical" (id 2) (at 148.59 66.04 0)
+      (effects (font (size 1.27 1.27)) hide)
+    )
+    (property "Datasheet" "~" (id 3) (at 148.59 66.04 0)
+      (effects (font (size 1.27 1.27)) hide)
+    )
+    (pin "1")
+    (pin "10")
+    (pin "2")
+    (pin "3")
+    (pin "4")
+    (pin "5")
+    (pin "6")
+    (pin "7")
+    (pin "8")
+    (pin "9")
+  )
 )

Commit message: schematic almost done
Parts:
- removed J?: PMOD, Connector_PinSocket_2.54mm:PinSocket_2x06_P2.54mm_Vertical, symbol Connector_Generic:Conn_02x06_Odd_Even
- removed J?: IDC_2x5, Connector_IDC:IDC-Header_2x05_P2.54mm_Vertical, symbol Connector_Generic:Conn_02x05_Odd_Even
- added J13: MINI_MOD_B, Connector_IDC:IDC-Header_2x05_P2.54mm_Vertical, symbol Connector_Generic:Conn_02x05_Odd_Even
- added J19: PMOD_I2C, Connector_PinSocket_2.54mm:PinSocket_2x04_P2.54mm_Vertical, symbol Connector_Generic:Conn_02x04_Odd_Even
- J11: renamed from J?; value IDC_2x10 -> EXT_MODULE
- J12: renamed from J?; value IDC_2x5 -> MINI_MOD_A
Connections:
- net +VDC: now reaches J11.1 (Pin_1)
- net +VDC: now also J11.2 (Pin_2), J12.1 (Pin_1), J13.1 (Pin_1)
- net EXT3: now reaches J11.10 (Pin_10)
- net EXT4: now reaches J11.11 (Pin_11)
- net EXT5: now reaches J11.12 (Pin_12)
- net EXT6: now reaches J11.13 (Pin_13)
- net EXT7: now reaches J11.14 (Pin_14)
- net EXT8: now reaches J11.15 (Pin_15)
- net EXT9: now reaches J11.16 (Pin_16)
- net EXT10: now reaches J11.17 (Pin_17)
- net EXT11: now reaches J11.18 (Pin_18)
- net EXT_SCL: now reaches J11.19 (Pin_19)
- net EXT_SDA: now reaches J11.20 (Pin_20)
- net +3V3: now reaches J11.3 (Pin_3)
- net +3V3: now also J11.4 (Pin_4), J12.2 (Pin_2), J13.2 (Pin_2), J19.7 (Pin_7), J19.8 (Pin_8)
- net GND: now reaches J11.5 (Pin_5)
- net GND: now also J11.6 (Pin_6), J12.3 (Pin_3), J13.3 (Pin_3), J19.5 (Pin_5), J19.6 (Pin_6)
- net EXT0: now reaches J11.7 (Pin_7)
- net EXT1: now reaches J11.8 (Pin_8)
- net EXT2: now reaches J11.9 (Pin_9)
- net MINI_A_SDA: now reaches J12.10 (Pin_10)
- net MINI_A_0: now reaches J12.4 (Pin_4)
- net MINI_A_1: now reaches J12.5 (Pin_5)
- net MINI_A_2: now reaches J12.6 (Pin_6)
- net MINI_A_3: now reaches J12.7 (Pin_7)
- net MINI_A_4: now reaches J12.8 (Pin_8)
- net MINI_A_SCL: now reaches J12.9 (Pin_9)
- new net MINI_B_0: J13.4 (Pin_4)
- new net MINI_B_1: J13.5 (Pin_5)
- new net MINI_B_2: J13.6 (Pin_6)
- new net MINI_B_3: J13.7 (Pin_7)
- new net MINI_B_4: J13.8 (Pin_8)
- new net MINI_B_SCL: J13.9 (Pin_9)
- new net MINI_B_SDA: J13.10 (Pin_10)
- new net PMOD_SCL: J19.1 (Pin_1), J19.2 (Pin_2)
- new net PMOD_SDA: J19.3 (Pin_3), J19.4 (Pin_4)
Other:
- note added: "Extension module connector"
- note added: "I2C PMOD-compatible socket"
- note added: "Mini module connector A"
- note added: "Mini module connector B"
- moved on the sheet: J11, J12

Commit message: routing done
Parts:
- added C31, C64: 4.7u 10V, Capacitor_SMD:C_0805_2012Metric, symbol Device:C_Small
- added F4, F5: 200mA SLOW, Fuse:Fuse_1206_3216Metric_Pad1.42x1.75mm_HandSolder, symbol Device:Fuse_Small
- added J2: POWER_OUT, TerminalBlock:TerminalBlock_bornier-2_P5.08mm, symbol Connector:Screw_Terminal_01x02
Connections:
- net +3V3: now also F4.2; no longer J12.2 (Pin_2), J13.2 (Pin_2)
- net +VDC: now also F5.2; no longer J12.1 (Pin_1), J13.1 (Pin_1)
- net GND: now also C31.2, C64.2, J2.2 (Pin_2)
- new net: C64.1, F5.1, J12.1 (Pin_1), J13.1 (Pin_1), J2.1 (Pin_1)
- new net: C31.1, F4.1, J12.2 (Pin_2), J13.2 (Pin_2)
Other:
- note added: "EXT POWER"
- moved on the sheet: J19

Commit message: schematics update
Other:
- company: (none) -> Wrocław University of Science and Technology
- title: (none) -> External connectors
Changed lines of the file:
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@@
 (kicad_sch (version 20211123) (generator eeschema)
   (paper "A4")
+  (title_block
+    (title "External connectors")
+    (date "2023-04-04")
+    (rev "1")
+    (company "Wrocław University of Science and Technology")
+    (comment 1 "Opensource educational robotic platform")
+    (comment 2 "Author: Jakub Mnich (jakub.mnich@pwr.edu.pl)")
+  )
   (junction (at 129.54 124.46) (diameter 0) (color 0 0 0 0)
   )
