File: line_sensors.kicad_sch (KiCad schematic)
At the start: 9 parts, among them U1 RPR-220, U2 RPR-220, U3 RPR-220, U4 RPR-220, U5 RPR-220, U6 RPR-220, U7 RPR-220, U8 RPR-220, U9 RPR-220

Commit message: Schematic in progress
Parts:
- added C? (x6): 100n 50V, Capacitor_SMD:C_0603_1608Metric, symbol Device:C_Small
- added R? (x9): 147R 1%, Resistor_SMD:R_0805_2012Metric_Pad1.20x1.40mm_HandSolder, symbol Device:R_Small
- added R? (x9): 3k3 1%, Resistor_SMD:R_0603_1608Metric_Pad0.98x0.95mm_HandSolder, symbol Device:R_Small
- added R?: 10k 1%, Resistor_SMD:R_0603_1608Metric_Pad0.98x0.95mm_HandSolder, symbol Device:R_Small
- added RV?: 100k POT, Potentiometer_SMD:Potentiometer_Bourns_3224W_Vertical, symbol Device:R_Potentiometer
- added U? (x15): LM393, Package_SO:SOIC-8_3.9x4.9mm_P1.27mm, symbol Comparator:LM393
- added U?: AP2171AW-7, Package_TO_SOT_SMD:SOT-23-5, symbol AP2171AW:AP2171AW-7
Connections:
- net at U3.1 (A): now also R?.2
- net GND: now reaches U3.2 (C)
- net GND: now also U1.2 (C), U1.3 (E), U2.2 (C), U2.3 (E), U3.3 (E), U4.2 (C), U4.3 (E), U5.2 (C), U5.3 (E), U6.2 (C), U6.3 (E), U7.2 (C), U7.3 (E), U8.2 (C), U8.3 (E), U9.2 (C), U9.3 (E), C?.2, C?.2, C?.2, C?.2, C?.2, C?.2, R?.2, RV?.3, U?.2 (GND), U?.4 (V-), U?.4 (V-), U?.4 (V-), U?.4 (V-), U?.4 (V-), U?.6 (_)
- net S3: now reaches U3.4 (C)
- net S3: now also R?.2, U?.2 (-)
- net at U9.1 (A): now also R?.2
- net S9: now reaches U9.4 (C)
- net S9: now also R?.2, U?.6 (_)
- net at U7.1 (A): now also R?.2
- net S7: now reaches U7.4 (C)
- net S7: now also R?.2, U?.6 (_)
- net at U8.1 (A): now also R?.2
- net S8: now reaches U8.4 (C)
- net S8: now also R?.2, U?.2 (-)
- net at U2.1 (A): now also R?.2
- net S2: now reaches U2.4 (C)
- net S2: now also R?.2, U?.6 (_)
- net at U1.1 (A): now also R?.2
- net S1: now reaches U1.4 (C)
- net S1: now also R?.2, U?.2 (-)
- net at U6.1 (A): now also R?.2
- net S6: now reaches U6.4 (C)
- net S6: now also R?.2, U?.2 (-)
- net at U4.1 (A): now also R?.2
- net S4: now reaches U4.4 (C)
- net S4: now also R?.2, U?.6 (_)
- net at U5.1 (A): now also R?.2
- net S5: now reaches U5.4 (C)
- net S5: now also R?.2, U?.2 (-)
- new net: R?.1, R?.1, R?.1, R?.1, R?.1, R?.1, R?.1, R?.1, R?.1, U?.1 (OUT)
- new net +3V3: C?.1, C?.1, C?.1, C?.1, C?.1, R?.1, R?.1, R?.1, R?.1, R?.1, R?.1, R?.1, R?.1, R?.1, RV?.1, U?.8 (V+), U?.8 (V+), U?.8 (V+), U?.8 (V+), U?.8 (V+)
- new net +VDC: U?.5 (IN)
- new net REF: C?.1, RV?.2, U?.3 (+), U?.3 (+), U?.3 (+), U?.3 (+), U?.3 (+), U?.5 (+), U?.5 (+), U?.5 (+), U?.5 (+), U?.5 (+)
- new net SENSOR_1: U?.1
- new net SENSOR_2: U?.7
- new net SENSOR_3: U?.1
- new net SENSOR_4: U?.7
- new net SENSOR_5: U?.1
- new net SENSOR_6: U?.1
- new net SENSOR_7: U?.7
- new net SENSOR_8: U?.1
- new net SENSOR_9: U?.7
- new net SEN_EN: R?.1, U?.4 (EN)
- no-connect marks 0 -> 2
Other:
- note added: "Comparators for line detection"
- note added: "Comparators' power supply"
- note added: "Detection threshold regulation"
- note added: "Reflective line sensors"
- moved on the sheet: U1, U2, U3, U4, U5, U6, U7, U8, U9

Commit message: schematic almost done
Parts:
- gave numbers to parts that had none: 32

Commit message: Layout in progress
Connections:
- net GND: now also U16.6 (_); no longer U18.6 (_)
- net S2: now also U17.2 (-); no longer U16.6 (_)
- net S3: now also U19.6 (_); no longer U17.2 (-)
- net S5: now also U19.2 (-); no longer U18.2 (-)
- net S6: now also U18.2 (-); no longer U19.2 (-)
- net S7: now also U20.2 (-); no longer U19.6 (_)
- net S8: now also U18.6 (_); no longer U20.2 (-)
Changed lines of the file:
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@@
-    (stroke (width 0) (type default) (color 0 0 0 0))
-  )
-  (wire (pts (xy 137.16 119.38) (xy 137.16 120.65))
     (stroke (width 0) (type default) (color 0 0 0 0))
   )
@@
   )
   (wire (pts (xy 50.8 101.6) (xy 58.42 101.6))
+    (stroke (width 0) (type default) (color 0 0 0 0))
+  )
+  (wire (pts (xy 50.8 119.38) (xy 50.8 120.65))
     (stroke (width 0) (type default) (color 0 0 0 0))
   )
@@
     (effects (font (size 2.5 2.5)) (justify left bottom))
   )
+  (label "REF" (at 224.79 101.6 0)
+    (effects (font (size 1.27 1.27)) (justify left bottom))
+  )
+  (label "REF" (at 93.98 114.3 0)
+    (effects (font (size 1.27 1.27)) (justify left bottom))
+  )
+  (label "S6" (at 194.31 46.99 0)
+    (effects (font (size 1.27 1.27)) (justify left bottom))
+  )
+  (label "S8" (at 247.65 46.99 0)
+    (effects (font (size 1.27 1.27)) (justify left bottom))
+  )
+  (label "S8" (at 137.16 119.38 0)
+    (effects (font (size 1.27 1.27)) (justify left bottom))
+  )
+  (label "REF" (at 93.98 101.6 0)
+    (effects (font (size 1.27 1.27)) (justify left bottom))
+  )
+  (label "S5" (at 167.64 46.99 0)
+    (effects (font (size 1.27 1.27)) (justify left bottom))
+  )
+  (label "S3" (at 114.3 46.99 0)
+    (effects (font (size 1.27 1.27)) (justify left bottom))
+  )
+  (label "S7" (at 224.79 106.68 0)
+    (effects (font (size 1.27 1.27)) (justify left bottom))
+  )
+  (label "S6" (at 137.16 106.68 0)
+    (effects (font (size 1.27 1.27)) (justify left bottom))
+  )
+  (label "REF" (at 50.8 114.3 0)
+    (effects (font (size 1.27 1.27)) (justify left bottom))
+  )
+  (label "S7" (at 220.98 46.99 0)
+    (effects (font (size 1.27 1.27)) (justify left bottom))
+  )
   (label "S1" (at 50.8 106.68 0)
     (effects (font (size 1.27 1.27)) (justify left bottom))
   )
-  (label "S3" (at 93.98 106.68 0)
-    (effects (font (size 1.27 1.27)) (justify left bottom))
-  )
-  (label "REF" (at 224.79 101.6 0)
-    (effects (font (size 1.27 1.27)) (justify left bottom))
-  )
-  (label "REF" (at 93.98 114.3 0)
-    (effects (font (size 1.27 1.27)) (justify left bottom))
-  )
-  (label "S6" (at 194.31 46.99 0)
-    (effects (font (size 1.27 1.27)) (justify left bottom))
-  )
-  (label "S8" (at 247.65 46.99 0)
-    (effects (font (size 1.27 1.27)) (justify left bottom))
-  )
-  (label "REF" (at 93.98 101.6 0)
-    (effects (font (size 1.27 1.27)) (justify left bottom))
-  )
-  (label "S5" (at 167.64 46.99 0)
-    (effects (font (size 1.27 1.27)) (justify left bottom))
-  )
-  (label "S3" (at 114.3 46.99 0)
-    (effects (font (size 1.27 1.27)) (justify left bottom))
-  )
-  (label "REF" (at 50.8 114.3 0)
-    (effects (font (size 1.27 1.27)) (justify left bottom))
-  )
-  (label "S7" (at 220.98 46.99 0)
-    (effects (font (size 1.27 1.27)) (justify left bottom))
-  )
-  (label "S6" (at 180.34 106.68 0)
+  (label "S3" (at 180.34 119.38 0)
     (effects (font (size 1.27 1.27)) (justify left bottom))
   )
@@
     (effects (font (size 1.27 1.27)) (justify left bottom))
   )
-  (label "S2" (at 50.8 119.38 0)
-    (effects (font (size 1.27 1.27)) (justify left bottom))
-  )
   (label "REF" (at 137.16 114.3 0)
     (effects (font (size 1.27 1.27)) (justify left bottom))
@@
     (effects (font (size 1.27 1.27)) (justify left bottom))
   )
-  (label "S8" (at 224.79 106.68 0)
+  (label "S5" (at 180.34 106.68 0)
     (effects (font (size 1.27 1.27)) (justify left bottom))
   )
@@
     (effects (font (size 1.27 1.27)) (justify left bottom))
   )
+  (label "S2" (at 93.98 106.68 0)
+    (effects (font (size 1.27 1.27)) (justify left bottom))
+  )
   (label "S9" (at 274.32 46.99 0)
     (effects (font (size 1.27 1.27)) (justify left bottom))
@@
     (effects (font (size 1.27 1.27)) (justify left bottom))
   )
-  (label "S5" (at 137.16 106.68 0)
-    (effects (font (size 1.27 1.27)) (justify left bottom))
-  )
   (label "S1" (at 60.96 46.99 0)
     (effects (font (size 1.27 1.27)) (justify left bottom))
@@
   )
   (label "REF" (at 180.34 114.3 0)
-    (effects (font (size 1.27 1.27)) (justify left bottom))
-  )
-  (label "S7" (at 180.34 119.38 0)
     (effects (font (size 1.27 1.27)) (justify left bottom))
   )
@@
     (pin "4")
     (pin "8")
-  )
-  (symbol (lib_id "power:GND") (at 137.16 120.65 0) (unit 1)
-    (in_bom yes) (on_board yes)
-    (property "Reference" "#PWR0103" (id 0) (at 137.16 127 0)
-      (effects (font (size 1.27 1.27)) hide)
-    )
-    (property "Value" "GND" (id 1) (at 137.16 124.46 0))
-    (property "Footprint" "" (id 2) (at 137.16 120.65 0)
-      (effects (font (size 1.27 1.27)) hide)
-    )
-    (property "Datasheet" "" (id 3) (at 137.16 120.65 0)
-      (effects (font (size 1.27 1.27)) hide)
-    )
-    (pin "1")
   )
   (symbol (lib_id "Device:R_Small") (at 265.43 45.72 0) (unit 1)
@@
     (pin "2")
   )
+  (symbol (lib_id "power:GND") (at 50.8 120.65 0) (unit 1)
+    (in_bom yes) (on_board yes)
+    (property "Reference" "#PWR?" (id 0) (at 50.8 127 0)
+      (effects (font (size 1.27 1.27)) hide)
+    )
+    (property "Value" "GND" (id 1) (at 50.8 124.46 0))
+    (property "Footprint" "" (id 2) (at 50.8 120.65 0)
+      (effects (font (size 1.27 1.27)) hide)
+    )
+    (property "Datasheet" "" (id 3) (at 50.8 120.65 0)
+      (effects (font (size 1.27 1.27)) hide)
+    )
+    (pin "1")
+  )
   (symbol (lib_id "Device:R_Small") (at 105.41 45.72 0) (unit 1)

Commit message: layout in progress
Connections:
- net S7: now also U20.6 (_); no longer U20.2 (-)
- net S9: now also U20.2 (-); no longer U20.6 (_)
- net SENSOR_2: now also U17.1; no longer U16.7
- net SENSOR_3: now also U19.7; no longer U17.1
- net SENSOR_5: now also U19.1; no longer U18.1
- net SENSOR_6: now also U18.1; no longer U19.1
- net SENSOR_7: now also U20.7; no longer U19.7
- net SENSOR_8: now also U18.7; no longer U20.1
- net SENSOR_9: now also U20.1; no longer U20.7
Changed lines of the file:
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@@
   )
   (no_connect (at 49.53 39.37))
-  (no_connect (at 162.56 116.84))
+  (no_connect (at 76.2 116.84))
   (wire (pts (xy 138.43 43.18) (xy 138.43 46.99))
     (stroke (width 0) (type default) (color 0 0 0 0))
@@
     (effects (font (size 1.27 1.27)) (justify left bottom))
   )
+  (label "S9" (at 224.79 106.68 0)
+    (effects (font (size 1.27 1.27)) (justify left bottom))
+  )
   (label "S5" (at 167.64 46.99 0)
     (effects (font (size 1.27 1.27)) (justify left bottom))
@@
     (effects (font (size 1.27 1.27)) (justify left bottom))
   )
-  (label "S7" (at 224.79 106.68 0)
-    (effects (font (size 1.27 1.27)) (justify left bottom))
-  )
   (label "S6" (at 137.16 106.68 0)
     (effects (font (size 1.27 1.27)) (justify left bottom))
@@
     (effects (font (size 1.27 1.27)) (justify left bottom))
   )
+  (label "S7" (at 224.79 119.38 0)
+    (effects (font (size 1.27 1.27)) (justify left bottom))
+  )
   (label "S9" (at 274.32 46.99 0)
-    (effects (font (size 1.27 1.27)) (justify left bottom))
-  )
-  (label "S9" (at 224.79 119.38 0)
     (effects (font (size 1.27 1.27)) (justify left bottom))
   )
@@
     (effects (font (size 1.27 1.27)) (justify left))
   )
-  (hierarchical_label "SENSOR_5" (shape output) (at 162.56 104.14 0)
+  (hierarchical_label "SENSOR_6" (shape output) (at 162.56 104.14 0)
     (effects (font (size 1.27 1.27)) (justify left))
   )
@@
     (effects (font (size 1.27 1.27)) (justify left))
   )
-  (hierarchical_label "SENSOR_9" (shape output) (at 250.19 116.84 0)
+  (hierarchical_label "SENSOR_7" (shape output) (at 250.19 116.84 0)
     (effects (font (size 1.27 1.27)) (justify left))
   )
-  (hierarchical_label "SENSOR_7" (shape output) (at 205.74 116.84 0)
+  (hierarchical_label "SENSOR_3" (shape output) (at 205.74 116.84 0)
     (effects (font (size 1.27 1.27)) (justify left))
   )
-  (hierarchical_label "SENSOR_6" (shape output) (at 205.74 104.14 0)
+  (hierarchical_label "SENSOR_5" (shape output) (at 205.74 104.14 0)
     (effects (font (size 1.27 1.27)) (justify left))
   )
-  (hierarchical_label "SENSOR_8" (shape output) (at 250.19 104.14 0)
+  (hierarchical_label "SENSOR_9" (shape output) (at 250.19 104.14 0)
     (effects (font (size 1.27 1.27)) (justify left))
   )
-  (hierarchical_label "SENSOR_3" (shape output) (at 119.38 104.14 0)
+  (hierarchical_label "SENSOR_8" (shape output) (at 162.56 116.84 0)
+    (effects (font (size 1.27 1.27)) (justify left))
+  )
+  (hierarchical_label "SENSOR_2" (shape output) (at 119.38 104.14 0)
     (effects (font (size 1.27 1.27)) (justify left))
   )
   (hierarchical_label "SEN_EN" (shape input) (at 26.67 39.37 180)
     (effects (font (size 1.27 1.27)) (justify right))
-  )
-  (hierarchical_label "SENSOR_2" (shape output) (at 76.2 116.84 0)
-    (effects (font (size 1.27 1.27)) (justify left))
   )
   (symbol (lib_id "power:+3.3V") (at 157.48 162.56 0) (unit 1)
@@
   (symbol (lib_id "power:GND") (at 50.8 120.65 0) (unit 1)
     (in_bom yes) (on_board yes)
-    (property "Reference" "#PWR?" (id 0) (at 50.8 127 0)
-      (effects (font (size 1.27 1.27)) hide)
-    )
+    (property "Reference" "#PWR0103" (id 0) (at 50.8 127 0)
+      (effects (font (size 1.27 1.27)) hide)
+    )

Commit message: schematics update
Other:
- company: (none) -> Wrocław University of Science and Technology
- title: (none) -> Line sensors
Changed lines of the file:
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@@
 (kicad_sch (version 20211123) (generator eeschema)
   (paper "A4")
+  (title_block
+    (title "Line sensors")
+    (date "2023-04-04")
+    (rev "1")
+    (company "Wrocław University of Science and Technology")
+    (comment 1 "Opensource educational robotic platform")
+    (comment 2 "Author: Jakub Mnich (jakub.mnich@pwr.edu.pl)")
+  )
   (junction (at 138.43 181.61) (diameter 0) (color 0 0 0 0)
   )
