File: power.kicad_sch (KiCad schematic)
At the start: 0 parts

Commit message: components selection
Parts:
- added BT1, BT2: LiION_18650, Battery:BatteryHolder_Keystone_1042_1x18650, symbol Device:Battery_Cell
- added C4, C6, C7: 100n 50V, Capacitor_SMD:C_0603_1608Metric, symbol Device:C_Small
- added C5, C8: 4.7u 10V, Capacitor_SMD:C_0805_2012Metric, symbol Device:C_Small
- added D1, D2: TVS, Diode_SMD:D_SMA, symbol Device:D_Zener_Small
- added D3: 5.1V, Diode_SMD:D_SMA, symbol Device:D_Zener_Small
- added D4: LED G, LED_SMD:LED_0603_1608Metric_Pad1.05x0.95mm_HandSolder, symbol Device:LED_Small
- added F1, F2: 5A SLOW, Fuse:Fuse_1206_3216Metric_Pad1.42x1.75mm_HandSolder, symbol Device:Fuse_Small
- added J1: Barrel_Jack, Connector_BarrelJack:BarrelJack_GCT_DCJ200-10-A_Horizontal, symbol Connector:Barrel_Jack
- added J2: BATTERY_OUT, TerminalBlock:TerminalBlock_bornier-2_P5.08mm, symbol Connector:Screw_Terminal_01x02
- added Q1, Q2, Q3: PMOS, Package_TO_SOT_SMD:TO-252-2, symbol Device:Q_PMOS_GDS
- added R2, R3: 1Meg 1%, Resistor_SMD:R_0603_1608Metric_Pad0.98x0.95mm_HandSolder, symbol Device:R_Small
- added R4, R5, R6, R8: 10k 1%, Resistor_SMD:R_0603_1608Metric_Pad0.98x0.95mm_HandSolder, symbol Device:R_Small
- added R7: 100R 1%, Resistor_SMD:R_0603_1608Metric_Pad0.98x0.95mm_HandSolder, symbol Device:R_Small
- added SW2: SW_SPDT, Button_Switch_THT:SW_Slide_1P2T_CK_OS102011MS2Q, symbol Switch:SW_SPDT
- added U12: AMS1117-3.3, Package_TO_SOT_SMD:SOT-223-3_TabPin2, symbol Regulator_Linear:AMS1117-3.3
Connections:
- new net: Q1.1 (G), R2.2, R4.1
- new net: D1.1 (K), F1.2, Q1.2 (D), R2.1
- new net: Q1.3 (S), Q2.3 (S), Q3.3 (S), R6.1
- new net: R7.2, SW2.2 (B), SW2.3 (C)
- new net: C4.1, Q3.1 (G), R6.2, R7.1
- new net: BT1.1 (+), F1.1
- new net: D4.2 (A), R8.1
- new net: Q2.1 (G), R3.2, R5.1
- new net: D2.1 (K), F2.2, Q2.2 (D), R3.1
- new net: BT2.1 (+), F2.1
- new net +3V3: C7.1, C8.1, U12.2 (VO)
- new net +BATT: C5.1, C6.1, J2.1 (Pin_1), Q3.2 (D), R8.2, U12.3 (VI)
- new net GND: BT1.2 (-), BT2.2 (-), C4.2, C5.2, C6.2, C7.2, C8.2, D1.2 (A), D2.2 (A), D4.1 (K), J2.2 (Pin_2), R4.2, R5.2, SW2.1 (A), U12.1 (GND)
Other:
- note added: "ADP2291ARMZ"

Commit message: working on the charger
Parts:
- added C?: 100n 50V, Capacitor_SMD:C_0603_1608Metric, symbol Device:C_Small
- added C?: 1u 10V, Capacitor_SMD:C_0603_1608Metric_Pad1.08x0.95mm_HandSolder, symbol Device:C_Small
- added C?: 10u 10V, Capacitor_SMD:C_0805_2012Metric, symbol Device:C_Small
- added D?: TVS, Diode_SMD:D_SMA, symbol Device:D_Zener_Small
- added D? (x4): 30V 5A, Diode_SMD:D_SOD-128, symbol Device:D_Zener_Small
- added D? (x2): 5.1V, Diode_SMD:D_SMA, symbol Device:D_Zener_Small
- added D?: ESDA6V1BC6, Package_TO_SOT_SMD:SOT-23-6, symbol Power_Protection:ESDA6V1BC6
- added D?: LED G, LED_SMD:LED_0603_1608Metric_Pad1.05x0.95mm_HandSolder, symbol Device:LED_Small
- added F?: 5A SLOW, Fuse:Fuse_1206_3216Metric_Pad1.42x1.75mm_HandSolder, symbol Device:Fuse_Small
- added J?: USB4085, GCT_USB4085:USB_C_Receptacle_GCT_USB4085, symbol Connector:USB_C_Receptacle_USB2.0
- added J?: CHG_IN, TerminalBlock:TerminalBlock_bornier-2_P5.08mm, symbol Connector:Screw_Terminal_01x02
- added Q? (x2): 2N7002NXAK, Package_TO_SOT_SMD:SOT-23, symbol Transistor_FET:2N7002
- added Q?: FZT549, Package_TO_SOT_SMD:SOT-223-3_TabPin2, symbol Device:Q_PNP_BCE
- added Q? (x2): PMOS, Package_TO_SOT_SMD:TO-252-2, symbol Device:Q_PMOS_GDS
- added Q?: NX3008PBK,215, Package_TO_SOT_SMD:SOT-23, symbol Device:Q_PMOS_GSD
- added R?: 1k5 5%, Resistor_SMD:R_0603_1608Metric_Pad0.98x0.95mm_HandSolder, symbol Device:R_Small
- added R? (x2): 5k1 1%, Resistor_SMD:R_0603_1608Metric_Pad0.98x0.95mm_HandSolder, symbol Device:R_Small
- added R? (x5): 10k 1%, Resistor_SMD:R_0603_1608Metric_Pad0.98x0.95mm_HandSolder, symbol Device:R_Small
- added R? (x4): 100R 1%, Resistor_SMD:R_0603_1608Metric_Pad0.98x0.95mm_HandSolder, symbol Device:R_Small
- added R? (x2): 0R, Resistor_SMD:R_0603_1608Metric_Pad0.98x0.95mm_HandSolder, symbol Device:R_Small
- added R?: 100k 1%, Resistor_SMD:R_0603_1608Metric_Pad0.98x0.95mm_HandSolder, symbol Device:R_Small
- added R?: 150m, Resistor_SMD:R_0805_2012Metric_Pad1.20x1.40mm_HandSolder, symbol Device:R_Small
- added U?: ADP2291, Package_SO:MSOP-8_3x3mm_P0.65mm, symbol ADP2291:ADP2291
- J1: M GCT -> Gravitech; MPN DCJ200-10-A-K1-K -> CON-SOCJ-2155
- J2: value BATTERY_OUT -> POWER_OUT
- SW2: value SW_SPDT -> OS102011MS2QN1
Connections:
- net GND: now also D3.2 (A), J1.2, C?.2, C?.2, C?.2, D?.2 (A), D?.2 (A), D?.2 (A), D?.2 (COM), D?.5 (COM), J?.1 (Pin_1), J?.A1 (GND), J?.A12 (GND), J?.B1 (GND), J?.B12 (GND), J?.S1 (SHIELD), Q?.2 (S), Q?.2 (S), R?.1, R?.1, R?.1, R?.1, R?.1, U?.2 (GND)
- net at Q1.3 (S), Q2.3 (S), Q3.3 (S)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: now also C?.1, Q?.2 (C), U?.3 (BAT)
- net at SW2.2 (B), SW2.3 (C): now also Q?.3 (D); no longer R7.2
- net at J1.1: now also F?.2, J?.2 (Pin_2)
- net at C4.1, Q3.1 (G), R6.2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: now also Q?.1 (G)
- net at D3.1 (K): now also Q?.1 (G), R?.1
- net +BATT renamed +VDC
- net +VDC: now also D?.1 (K), D?.1 (K), Q?.3 (S); no longer Q3.2 (D)
- new net: Q?.1 (G), R?.2
- new net: Q?.3 (D), R?.1
- new net: D?.1 (K), Q?.1 (G), R?.1 (x2)
- new net: Q?.3 (D), R?.1, R?.1
- new net: J?.A5 (CC1), R?.2
- new net: D?.2 (A), D?.2 (A), Q?.2 (D)
- new net: D?.1 (TVS1), D?.3 (TVS2), J?.A6 (D+), J?.B6 (D+), R?.1
- new net: D?.4 (TVS3), D?.6 (TVS4), J?.A7 (D-), J?.B7 (D-), R?.1
- new net: J?.B5 (CC2), R?.2
- new net: Q?.2 (S), R7.2
- new net: Q?.1 (B), U?.1 (DRV)
- new net: Q?.3 (E), R?.1, U?.4 (CS)
- new net: Q3.2 (D), Q?.2 (D)
- new net: D?.2 (A), R?.1
- new net: R?.2, U?.5 (ADJ)
- new net: C?.1, U?.7 (TIMER)
- new net: D?.1 (K), U?.8 (CHG)
- new net CHARGE_POW_INPUT: D?.1 (K), D?.1 (K), R?.2, R?.2, R?.2, R?.2, U?.6 (IN)
- new net CHARGING_BUS_RAW: D?.1 (K), D?.2 (A), D?.2 (A), F?.1, R?.2, R?.2, R?.2, R?.2
- new net DM: R?.2
- new net DP: R?.1, R?.2
- new net DP_PULL: R?.2
- new net VBUS: C?.1, J?.A4 (VBUS), J?.A9 (VBUS), J?.B4 (VBUS), J?.B9 (VBUS), Q?.3 (S), R?.2
- no-connect marks 0 -> 2
Other:
- note added: "CHARGING CURRENT ADJUSTEMENT WITH ADJ PIN: FLOAT - 1125 mA 100K PULL - 375 mA"
- note removed: "ADP2291ARMZ"
- moved on the sheet: BT1, BT2, C4, C5, C6, C7, C8, D1, D2, D3, D4, F1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

Commit message: Schematic in progress
Parts:
- removed D1, D2: TVS, Diode_SMD:D_SMA, symbol Device:D_Zener_Small
- added C11, C13, C?: 100n 50V, Capacitor_SMD:C_0603_1608Metric, symbol Device:C_Small
- added R20, R21: 100k 1%, Resistor_SMD:R_0603_1608Metric_Pad0.98x0.95mm_HandSolder, symbol Device:R_Small
- added U14: MCP6006R, Package_TO_SOT_SMD:SOT-23-5, symbol AD8541ARTZ:AD8541ARTZ
- gave numbers to parts that had none: 38
Connections:
- net +3V3: now also C13.1, U14.2 (V+)
- net +VDC: now also R20.1
- net GND: now also C11.2, C13.2, C?.2, R21.2, U14.5 (V-)
- net VBUS: now also C?.1
- net CHARGING_BUS_RAW renamed BARREL_JACK_BUS
- net DM renamed USB_DM
- net DP renamed USB_DP
- net DP_PULL renamed USB_DP_PULL
- new net: C11.1, R20.2, R21.1, U14.3 (+)
- new net VOLTAGE_MONITOR: U14.1, U14.4 (-)
Other:
- note added: "3V3 bus regulator"
- note added: "AUTOMATIC CHARGING CURRENT ADJUSTEMENT: EXTERNAL POWER - 1125 mA VBUS POWER - 375 mA"
- note added: "Batteries"
- note added: "Battery charger"
- note added: "External power connection"
- note added: "Main bus voltage measurement"
- note added: "Main power switch"
- note added: "USB Connector"
- note added: "VBUS cutoff"
- note removed: "CHARGING CURRENT ADJUSTEMENT WITH ADJ PIN: FLOAT - 1125 mA 100K PULL - 375 mA"
- moved on the sheet: BT1, BT2, C10, C12, C4, C5, C6, C7, C8, C9, D10, D11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

Commit message: schematic almost done
Parts:
- U12: value AMS1117-3.3 -> TC1108-3.3; M TI -> Microchip; MPN LM1117MPX-3.3/NOPB -> TC1108-3.3VDBTR
- gave numbers to parts that had none: 1
Connections:
- net +3V3: now also U12.3 (VO); no longer U12.2 (VO)
- net +VDC: now also U12.1 (VI); no longer U12.3 (VI)
- net GND: now also U12.2 (GND); no longer U12.1 (GND)
Changed lines of the file:
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@@
   (symbol (lib_id "power:VBUS") (at 259.08 106.68 0) (unit 1)
     (in_bom yes) (on_board yes)
-    (property "Reference" "#PWR?" (id 0) (at 259.08 110.49 0)
+    (property "Reference" "#PWR0196" (id 0) (at 259.08 110.49 0)
       (effects (font (size 1.27 1.27)) hide)
     )
@@
   (symbol (lib_id "Device:C_Small") (at 259.08 110.49 0) (unit 1)
     (in_bom yes) (on_board yes)
-    (property "Reference" "C?" (id 0) (at 260.35 107.95 0)
+    (property "Reference" "C52" (id 0) (at 260.35 107.95 0)
       (effects (font (size 1.27 1.27)) (justify left))
     )
@@
     (in_bom yes) (on_board yes)
     (property "Reference" "U12" (id 0) (at 232.41 24.13 0))
-    (property "Value" "AMS1117-3.3" (id 1) (at 237.49 26.67 0))
+    (property "Value" "TC1108-3.3" (id 1) (at 237.49 26.67 0))
     (property "Footprint" "Package_TO_SOT_SMD:SOT-223-3_TabPin2" (id 2) (at 237.49 25.4 0)
       (effects (font (size 1.27 1.27)) hide)
     )
-    (property "Datasheet" "http://www.advanced-monolithic.com/pdf/ds1117.pdf" (id 3) (at 240.03 36.83 0)
-      (effects (font (size 1.27 1.27)) hide)
-    )
-    (property "M" "TI" (id 4) (at 237.49 30.48 0)
-      (effects (font (size 1.27 1.27)) hide)
-    )
-    (property "MPN" "LM1117MPX-3.3/NOPB" (id 5) (at 237.49 30.48 0)
-      (effects (font (size 1.27 1.27)) hide)
-    )
-    (pin "1")
+    (property "Datasheet" "https://www.mouser.pl/datasheet/2/268/MCHPS04200_1-2520760.pdf" (id 3) (at 240.03 38.1 0)
+      (effects (font (size 1.27 1.27)) hide)
+    )
+    (property "M" "Microchip" (id 4) (at 237.49 26.67 0)
+      (effects (font (size 1.27 1.27)) hide)
+    )
+    (property "MPN" "TC1108-3.3VDBTR" (id 5) (at 238.76 25.4 0)
+      (effects (font (size 1.27 1.27)) hide)
+    )
     (pin "2")
     (pin "3")
+    (pin "1")
   )
   (symbol (lib_id "power:GND") (at 55.88 189.23 0) (unit 1)
@@
   (symbol (lib_id "power:GND") (at 259.08 114.3 0) (unit 1)
     (in_bom yes) (on_board yes)
-    (property "Reference" "#PWR?" (id 0) (at 259.08 120.65 0)
-      (effects (font (size 1.27 1.27)) hide)
-    )
+    (property "Reference" "#PWR0197" (id 0) (at 259.08 120.65 0)
+      (effects (font (size 1.27 1.27)) hide)
+    )

Commit message: routing done
Parts:
- removed J2: POWER_OUT, TerminalBlock:TerminalBlock_bornier-2_P5.08mm, symbol Connector:Screw_Terminal_01x02
Changed lines of the file:
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@@
-    (stroke (width 0) (type default) (color 0 0 0 0))
-  )
-  (wire (pts (xy 111.76 95.25) (xy 113.03 95.25))
     (stroke (width 0) (type default) (color 0 0 0 0))
   )
@@
     (stroke (width 0) (type default) (color 0 0 0 0))
   )
-  (wire (pts (xy 111.76 99.06) (xy 111.76 97.79))
-    (stroke (width 0) (type default) (color 0 0 0 0))
-  )
   (wire (pts (xy 85.09 85.09) (xy 85.09 87.63))
     (stroke (width 0) (type default) (color 0 0 0 0))
@@
     (stroke (width 0) (type default) (color 0 0 0 0))
   )
-  (wire (pts (xy 111.76 97.79) (xy 113.03 97.79))
-    (stroke (width 0) (type default) (color 0 0 0 0))
-  )
   (wire (pts (xy 135.89 36.83) (xy 139.7 36.83))
     (stroke (width 0) (type default) (color 0 0 0 0))
@@
   )
   (wire (pts (xy 204.47 76.2) (xy 204.47 80.01))
-    (stroke (width 0) (type default) (color 0 0 0 0))
-  )
-  (wire (pts (xy 111.76 93.98) (xy 111.76 95.25))
     (stroke (width 0) (type default) (color 0 0 0 0))
   )
@@
     )
     (property "Datasheet" "" (id 3) (at 220.98 40.64 0)
-      (effects (font (size 1.27 1.27)) hide)
-    )
-    (pin "1")
-  )
-  (symbol (lib_id "power:+VDC") (at 111.76 93.98 0) (unit 1)
-    (in_bom yes) (on_board yes) (fields_autoplaced)
-    (property "Reference" "#PWR041" (id 0) (at 111.76 96.52 0)
-      (effects (font (size 1.27 1.27)) hide)
-    )
-    (property "Value" "+VDC" (id 1) (at 111.76 86.36 0))
-    (property "Footprint" "" (id 2) (at 111.76 93.98 0)
-      (effects (font (size 1.27 1.27)) hide)
-    )
-    (property "Datasheet" "" (id 3) (at 111.76 93.98 0)
       (effects (font (size 1.27 1.27)) hide)
     )
@@
     (pin "8")
   )
-  (symbol (lib_id "Connector:Screw_Terminal_01x02") (at 118.11 95.25 0) (unit 1)
-    (in_bom yes) (on_board yes)
-    (property "Reference" "J2" (id 0) (at 115.57 92.71 0)
-      (effects (font (size 1.27 1.27)) (justify left))
-    )
-    (property "Value" "POWER_OUT" (id 1) (at 121.92 102.87 90)
-      (effects (font (size 1.27 1.27)) (justify left))
-    )
-    (property "Footprint" "TerminalBlock:TerminalBlock_bornier-2_P5.08mm" (id 2) (at 118.11 95.25 0)
-      (effects (font (size 1.27 1.27)) hide)
-    )
-    (property "Datasheet" "~" (id 3) (at 118.11 95.25 0)
-      (effects (font (size 1.27 1.27)) hide)
-    )
-    (pin "1")
-    (pin "2")
-  )
   (symbol (lib_id "Device:Fuse_Small") (at 44.45 41.91 180) (unit 1)
     (in_bom yes) (on_board yes)
@@
     (pin "2")
   )
-  (symbol (lib_id "power:GND") (at 111.76 99.06 0) (unit 1)
-    (in_bom yes) (on_board yes)
-    (property "Reference" "#PWR021" (id 0) (at 111.76 105.41 0)
-      (effects (font (size 1.27 1.27)) hide)
-    )
-    (property "Value" "GND" (id 1) (at 111.76 102.87 0))
-    (property "Footprint" "" (id 2) (at 111.76 99.06 0)
-      (effects (font (size 1.27 1.27)) hide)
-    )
-    (property "Datasheet" "" (id 3) (at 111.76 99.06 0)
-      (effects (font (size 1.27 1.27)) hide)
-    )
-    (pin "1")
-  )
   (symbol (lib_id "Device:Fuse_Small") (at 55.88 128.27 90) (unit 1)

Commit message: schematics update
Other:
- company: (none) -> Wrocław University of Science and Technology
- title: (none) -> Power system and USB-C connector
Changed lines of the file:
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@@
 (kicad_sch (version 20211123) (generator eeschema)
   (paper "A4")
+  (title_block
+    (title "Power system and USB-C connector")
+    (date "2023-04-04")
+    (rev "1")
+    (company "Wrocław University of Science and Technology")
+    (comment 1 "Opensource educational robotic platform")
+    (comment 2 "Author: Jakub Mnich (jakub.mnich@pwr.edu.pl)")
+  )
   (junction (at 66.04 41.91) (diameter 0) (color 0 0 0 0)
   )
