File: structural.kicad_sch (KiCad schematic)
At the start: 15 parts

Commit message: Layout in progress
Parts:
- removed H1, H6: Caster_hole, MountingHole:MountingHole_2.2mm_M2_DIN965_Pad, symbol Mechanical:MountingHole
- removed H10, H4, H5, H9: Interface_hole, MountingHole:MountingHole_3.2mm_M3_DIN965_Pad, symbol Mechanical:MountingHole
- removed H11, H12, H13, H14, H15: Bumper_hole, MountingHole:MountingHole_3.2mm_M3_DIN965_Pad, symbol Mechanical:MountingHole
- removed H2, H3, H7, H8: Motor_hole, MountingHole:MountingHole_3.2mm_M3_DIN965_Pad, symbol Mechanical:MountingHole
- added H1, H6: Caster_hole, MountingHole:MountingHole_2.2mm_M2_DIN965_Pad, symbol Mechanical:MountingHole_Pad
- added H10, H4, H5, H9: Interface_hole, MountingHole:MountingHole_3.2mm_M3_DIN965_Pad, symbol Mechanical:MountingHole_Pad
- added H11, H12, H13, H14, H15: Bumber_hole, MountingHole:MountingHole_3.2mm_M3_DIN965_Pad, symbol Mechanical:MountingHole_Pad
- added H2, H3, H7, H8: Motor_hole, MountingHole:MountingHole_3.2mm_M3_DIN965_Pad, symbol Mechanical:MountingHole_Pad
Connections:
- new net GND: H1.1, H10.1, H11.1, H12.1, H13.1, H14.1, H15.1, H2.1, H3.1, H4.1, H5.1, H6.1, H7.1, H8.1, H9.1

Commit message: schematics update
Other:
- company: (none) -> Wrocław University of Science and Technology
- title: (none) -> Structural holes
Changed lines of the file:
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@@
 (kicad_sch (version 20211123) (generator eeschema)
   (paper "A4")
+  (title_block
+    (title "Structural holes")
+    (date "2023-04-04")
+    (rev "1")
+    (company "Wrocław University of Science and Technology")
+    (comment 1 "Opensource educational robotic platform")
+    (comment 2 "Author: Jakub Mnich (jakub.mnich@pwr.edu.pl)")
+  )
   (symbol (lib_id "Mechanical:MountingHole_Pad") (at 93.98 102.87 0) (unit 1)
     (in_bom yes) (on_board yes) (fields_autoplaced)
